File: fan.kicad_pcb (KiCad board)
At the start: 2 copper layers, 297.2 x 263.7 mm, 192 parts, among them J1 01x04_Male, J2 Pi, SW1 SW_PUSH, SW10 SW_PUSH, SW11 SW_PUSH, SW12 SW_PUSH, SW13 SW_PUSH, SW14 SW_PUSH, SW15 SW_PUSH, SW16 SW_PUSH, SW17 SW_PUSH, SW18 SW_PUSH, SW19 SW_PUSH, SW2 SW_PUSH, SW20 SW_PUSH, SW21 SW_PUSH, SW22 SW_PUSH, SW23 SW_PUSH, SW24 SW_PUSH, SW25 SW_PUSH, SW26 SW_PUSH, SW27 SW_PUSH, SW28 SW_PUSH, SW29 SW_PUSH, SW3 SW_PUSH, SW30 SW_PUSH, SW31 SW_PUSH, SW32 SW_PUSH, SW33 SW_PUSH, SW34 SW_PUSH, SW35 SW_PUSH, SW36 SW_PUSH, SW37 SW_PUSH, SW38 SW_PUSH, SW39 SW_PUSH, SW4 SW_PUSH, SW40 SW_PUSH, SW41 SW_PUSH, SW42 SW_PUSH, SW43 SW_PUSH, SW44 SW_PUSH, SW45 SW_PUSH, SW46 SW_PUSH, SW47 SW_PUSH, SW48 SW_PUSH, SW49 SW_PUSH, SW5 SW_PUSH, SW50 SW_PUSH, SW51 SW_PUSH, SW52 SW_PUSH, SW53 SW_PUSH, SW54 SW_PUSH, SW55 SW_PUSH, SW56 SW_PUSH, SW57 SW_PUSH, SW58 SW_PUSH, SW59 SW_PUSH, SW6 SW_PUSH, SW60 SW_PUSH, SW61 SW_PUSH, SW62 SW_PUSH, SW63 SW_PUSH, SW64 SW_PUSH, SW65 SW_PUSH, SW66 SW_PUSH, SW67 SW_PUSH, SW68 SW_PUSH, SW69 SW_PUSH, SW7 SW_PUSH, SW70 SW_PUSH, SW71 SW_PUSH, SW72 SW_PUSH, SW73 SW_PUSH, SW74 SW_PUSH, SW75 SW_PUSH, SW76 SW_PUSH, SW77 SW_PUSH, SW78 SW_PUSH, SW79 SW_PUSH, SW8 SW_PUSH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

Commit message: pro microに変更
Parts:
- removed A1, A2: Arduino_Nano_v2.x, Module:Arduino_Nano
- removed J1: 01x04_Male, Connector_PinSocket_2.54mm:PinSocket_1x04_P2.54mm_Vertical
- removed the Ref** at (128.0, 282.6)
- removed the Ref** at (274.2, 359.1)
- removed the Ref** at (119.6, 143.2)
- removed the Ref** at (296.1, 130.2)
- removed the Ref** at (235.8, 263.8)
- removed the Ref** at (390.4, 294.8)
- added Ref**: Val**, kbd:HOLE, F.Cu at (236.2, 264.4)
- added Ref**: Val**, kbd:HOLE, F.Cu at (128.0, 284.0)
- added Ref**: Val**, kbd:HOLE, F.Cu at (273.6, 359.2)
- added Ref**: Val**, kbd:HOLE, F.Cu at (390.4, 294.8)
- added Ref**: Val**, kbd:HOLE, F.Cu at (286.4, 147.4)
- added Ref**: Val**, kbd:HOLE, F.Cu at (118.4, 143.0)
- added SW93: SW_SPDT, Button_Switch_THT:SW_Slide_1P2T_CK_OS102011MS2Q, F.Cu at (295.5, 152.8)
- added U1: ProMicro, kbd:ProMicro_v3.5, F.Cu at (188.9, 121.9)
- added U2: ProMicro, kbd:ProMicro_v3.5, B.Cu at (190.2, 118.8)
- added U3: 74HC595, digikey-footprints:DIP-16_W7.62mm, F.Cu at (211.8, 127.0)
- added U4: 74HC595, digikey-footprints:DIP-16_W7.62mm, F.Cu at (233.8, 129.2)
- moved SW92 19.4 mm to (226.9, 115.3), turned to 174 degrees
- moved SW91 9.68 mm to (238.2, 116.5), turned to 174 degrees
- moved J2 3.45 mm to (263.4, 124.4)
Connections:
- net VCC renamed Net-(J2-Pad38)
- SW91 pad 1: reset -> software_reset
- SW92 pad 1: reset_arduino -> hardware_reset
Routing:
- net VCC: track 0.00 -> 165.7 mm, vias 0 -> 1
- net Net-(J2-Pad38): track 125.1 -> 14.2 mm, vias 1 -> 0
- net 3V: track 86.9 -> 0.00 mm
- net GND: track 81.7 -> 0.00 mm
- net SCK: track 0.00 -> 73.3 mm, vias 0 -> 2
- net SCL: track 0.00 -> 67.8 mm, vias 0 -> 1
- net software_reset: track 0.00 -> 66.9 mm, vias 0 -> 1
- net hardware_reset: track 0.00 -> 66.6 mm
- net RCK: track 0.00 -> 62.3 mm, vias 0 -> 2
- net col10: track 524.9 -> 462.9 mm, vias 6 -> 7
- net 5V: track 60.2 -> 0.00 mm
- net OE: track 0.00 -> 59.9 mm, vias 0 -> 2
- net col14: track 531.7 -> 472.6 mm
- net col05: track 350.6 -> 293.8 mm, vias 6 -> 5
- net col09: track 411.4 -> 357.4 mm, vias 4 -> 5
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