File: fan.sch (KiCad schematic (older format))
At the start: 186 parts, among them J1 01x04_Male, J2 Pi, SW1 SW_PUSH, SW10 SW_PUSH, SW11 SW_PUSH, SW12 SW_PUSH, SW13 SW_PUSH, SW14 SW_PUSH, SW15 SW_PUSH, SW16 SW_PUSH, SW17 SW_PUSH, SW18 SW_PUSH, SW19 SW_PUSH, SW2 SW_PUSH, SW20 SW_PUSH, SW21 SW_PUSH, SW22 SW_PUSH, SW23 SW_PUSH, SW24 SW_PUSH, SW25 SW_PUSH, SW26 SW_PUSH, SW27 SW_PUSH, SW28 SW_PUSH, SW29 SW_PUSH, SW3 SW_PUSH, SW30 SW_PUSH, SW31 SW_PUSH, SW32 SW_PUSH, SW33 SW_PUSH, SW34 SW_PUSH, SW35 SW_PUSH, SW36 SW_PUSH, SW37 SW_PUSH, SW38 SW_PUSH, SW39 SW_PUSH, SW4 SW_PUSH, SW40 SW_PUSH, SW41 SW_PUSH, SW42 SW_PUSH, SW43 SW_PUSH, SW44 SW_PUSH, SW45 SW_PUSH, SW46 SW_PUSH, SW47 SW_PUSH, SW48 SW_PUSH, SW49 SW_PUSH, SW5 SW_PUSH, SW50 SW_PUSH, SW51 SW_PUSH, SW52 SW_PUSH, SW53 SW_PUSH, SW54 SW_PUSH, SW55 SW_PUSH, SW56 SW_PUSH, SW57 SW_PUSH, SW58 SW_PUSH, SW59 SW_PUSH, SW6 SW_PUSH, SW60 SW_PUSH, SW61 SW_PUSH, SW62 SW_PUSH, SW63 SW_PUSH, SW64 SW_PUSH, SW65 SW_PUSH, SW66 SW_PUSH, SW67 SW_PUSH, SW68 SW_PUSH, SW69 SW_PUSH, SW7 SW_PUSH, SW70 SW_PUSH, SW71 SW_PUSH, SW72 SW_PUSH, SW73 SW_PUSH, SW74 SW_PUSH, SW75 SW_PUSH, SW76 SW_PUSH, SW77 SW_PUSH, SW78 SW_PUSH, SW79 SW_PUSH, SW8 SW_PUSH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

Commit message: pro microに変更
Parts:
- removed A1, A2: Arduino_Nano_v2.x, Module:Arduino_Nano, symbol MCU_Module:Arduino_Nano_v2.x
- removed J1: 01x04_Male, Connector_PinSocket_2.54mm:PinSocket_1x04_P2.54mm_Vertical, symbol Connector:Conn_01x04_Male
- added SW93: SW_SPDT, Button_Switch_THT:SW_Slide_1P2T_CK_OS102011MS2Q, symbol Switch:SW_SPDT
- added U1, U2: ProMicro, kbd:ProMicro_v3.5, symbol kbd:ProMicro
- added U3, U4: 74HC595, digikey-footprints:DIP-16_W7.62mm, symbol 74xx:74HC595
Connections:
- net GND: now also U1.23 (GND), U1.3 (GND), U1.4 (GND), U2.23 (GND), U2.3 (GND), U2.4 (GND), U3.8 (GND), U4.8 (GND)
- net VCC: now also SW93.3 (C), U1.21 (VCC), U2.21 (VCC), U3.16 (VCC), U4.16 (VCC); no longer J2.38 (Pin_38), J2.40 (Pin_40)
- net col00: now also U3.15 (QA)
- net col01: now also U3.1 (QB)
- net col02: now also U3.2 (QC)
- net col03: now also U3.3 (QD)
- net col04: now also U3.4 (QE)
- net col05: now also U3.5 (QF)
- net col06: now also U3.6 (QG)
- net col07: now also U3.7 (QH)
- net col08: now also U4.15 (QA)
- net col09: now also U4.1 (QB)
- net col10: now also U4.2 (QC)
- net col11: now also U4.3 (QD)
- net col12: now also U4.4 (QE)
- net col13: now also U4.5 (QF)
- net col14: now also U4.6 (QG)
- net row00: now also U1.18 (F6/A1), U2.18 (F6/A1)
- net row01: now also U1.17 (F7/A0), U2.17 (F7/A0)
- net row02: now also U1.16 (B1/15), U2.16 (B1/15)
- net row03: now also U1.15 (B3/14), U2.15 (B3/14)
- net row04: now also U1.14 (B2/16), U2.14 (B2/16)
- net row05: now also U1.13 (B6/10), U2.13 (B6/10)
- net reset renamed software_reset
- net software_reset: now also U1.7 (4/D4), U2.7 (4/D4)
- net reset_arduino renamed hardware_reset
- net hardware_reset: now also U1.22 (RST), U2.22 (RST)
- new net: U3.9 (QH'), U4.14 (SER)
- new net: J2.38 (Pin_38), J2.40 (Pin_40), SW93.2 (B)
- new net OE: U1.12 (9/B5), U2.12 (9/B5), U3.13 (~OE), U4.13 (~OE)
- new net RCK: U1.11 (8/B4), U2.11 (8/B4), U3.12 (RCLK), U4.12 (RCLK)
- new net SCK: U1.9 (6/D7), U2.9 (6/D7), U3.11 (SRCLK), U4.11 (SRCLK)
- new net SCL: U1.10 (7/E6), U2.10 (7/E6), U3.10 (~SRCLR), U4.10 (~SRCLR)
- new net SER: U1.8 (5/C6), U2.8 (5/C6), U3.14 (SER)
- no-connect marks 42 -> 57
Other:
- moved on the sheet: J2, SW91, SW92
