File: fan/fan.sch (KiCad schematic (older format))
At the start: 190 parts, among them J2 Pi, SW1 SW_PUSH, SW10 SW_PUSH, SW11 SW_PUSH, SW12 SW_PUSH, SW13 SW_PUSH, SW14 SW_PUSH, SW15 SW_PUSH, SW16 SW_PUSH, SW17 SW_PUSH, SW18 SW_PUSH, SW19 SW_PUSH, SW2 SW_PUSH, SW20 SW_PUSH, SW21 SW_PUSH, SW22 SW_PUSH, SW23 SW_PUSH, SW24 SW_PUSH, SW25 SW_PUSH, SW26 SW_PUSH, SW27 SW_PUSH, SW28 SW_PUSH, SW29 SW_PUSH, SW3 SW_PUSH, SW30 SW_PUSH, SW31 SW_PUSH, SW32 SW_PUSH, SW33 SW_PUSH, SW34 SW_PUSH, SW35 SW_PUSH, SW36 SW_PUSH, SW37 SW_PUSH, SW38 SW_PUSH, SW39 SW_PUSH, SW4 SW_PUSH, SW40 SW_PUSH, SW41 SW_PUSH, SW42 SW_PUSH, SW43 SW_PUSH, SW44 SW_PUSH, SW45 SW_PUSH, SW46 SW_PUSH, SW47 SW_PUSH, SW48 SW_PUSH, SW49 SW_PUSH, SW5 SW_PUSH, SW50 SW_PUSH, SW51 SW_PUSH, SW52 SW_PUSH, SW53 SW_PUSH, SW54 SW_PUSH, SW55 SW_PUSH, SW56 SW_PUSH, SW57 SW_PUSH, SW58 SW_PUSH, SW59 SW_PUSH, SW6 SW_PUSH, SW60 SW_PUSH, SW61 SW_PUSH, SW62 SW_PUSH, SW63 SW_PUSH, SW64 SW_PUSH, SW65 SW_PUSH, SW66 SW_PUSH, SW67 SW_PUSH, SW68 SW_PUSH, SW69 SW_PUSH, SW7 SW_PUSH, SW70 SW_PUSH, SW71 SW_PUSH, SW72 SW_PUSH, SW73 SW_PUSH, SW74 SW_PUSH, SW75 SW_PUSH, SW76 SW_PUSH, SW77 SW_PUSH, SW78 SW_PUSH, SW79 SW_PUSH, SW8 SW_PUSH, SW80 SW_PUSH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

Commit message: 大幅に手戻り 配線最初から
Connections:
- net QHSER: no longer U5.9 (QH'), U6.14 (SER)
- net row00: now also D13.2 (K), D19.2 (K), D25.2 (K), D31.2 (K), D37.2 (K), D43.2 (K), D49.2 (K), D55.2 (K), D61.2 (K), D67.2 (K), D7.2 (K), D73.2 (K), D79.2 (K), D85.2 (K); no longer D13.1 (A), D19.1 (A), D25.1 (A), D31.1 (A), D37.1 (A), D43.1 (A), D49.1 (A), D55.1 (A), D61.1 (A), D67.1 (A), D7.1 (A), D73.1 (A), D79.1 (A), D85.1 (A)
- net row01: now also D14.2 (K), D2.2 (K), D20.2 (K), D26.2 (K), D32.2 (K), D38.2 (K), D44.2 (K), D50.2 (K), D56.2 (K), D62.2 (K), D68.2 (K), D74.2 (K), D8.2 (K), D80.2 (K), D86.2 (K); no longer D14.1 (A), D2.1 (A), D20.1 (A), D26.1 (A), D32.1 (A), D38.1 (A), D44.1 (A), D50.1 (A), D56.1 (A), D62.1 (A), D68.1 (A), D74.1 (A), D8.1 (A), D80.1 (A), D86.1 (A)
- net row02: now also D15.2 (K), D21.2 (K), D27.2 (K), D3.2 (K), D33.2 (K), D39.2 (K), D45.2 (K), D51.2 (K), D57.2 (K), D63.2 (K), D69.2 (K), D75.2 (K), D81.2 (K), D87.2 (K), D9.2 (K); no longer D15.1 (A), D21.1 (A), D27.1 (A), D3.1 (A), D33.1 (A), D39.1 (A), D45.1 (A), D51.1 (A), D57.1 (A), D63.1 (A), D69.1 (A), D75.1 (A), D81.1 (A), D87.1 (A), D9.1 (A)
- net row03: now also D10.2 (K), D16.2 (K), D22.2 (K), D28.2 (K), D34.2 (K), D4.2 (K), D40.2 (K), D46.2 (K), D52.2 (K), D58.2 (K), D64.2 (K), D70.2 (K), D76.2 (K), D82.2 (K), D88.2 (K); no longer D10.1 (A), D16.1 (A), D22.1 (A), D28.1 (A), D34.1 (A), D4.1 (A), D40.1 (A), D46.1 (A), D52.1 (A), D58.1 (A), D64.1 (A), D70.1 (A), D76.1 (A), D82.1 (A), D88.1 (A)
- net row04: now also D11.2 (K), D17.2 (K), D23.2 (K), D29.2 (K), D35.2 (K), D41.2 (K), D47.2 (K), D5.2 (K), D53.2 (K), D59.2 (K), D71.2 (K), D77.2 (K), D83.2 (K), D89.2 (K); no longer D11.1 (A), D17.1 (A), D23.1 (A), D29.1 (A), D35.1 (A), D41.1 (A), D47.1 (A), D5.1 (A), D53.1 (A), D59.1 (A), D71.1 (A), D77.1 (A), D83.1 (A), D89.1 (A)
- net row05: now also D12.2 (K), D18.2 (K), D24.2 (K), D30.2 (K), D36.2 (K), D42.2 (K), D48.2 (K), D54.2 (K), D6.2 (K), D60.2 (K), D66.2 (K), D72.2 (K), D78.2 (K), D84.2 (K), D90.2 (K); no longer D12.1 (A), D18.1 (A), D24.1 (A), D30.1 (A), D36.1 (A), D42.1 (A), D48.1 (A), D54.1 (A), D6.1 (A), D60.1 (A), D66.1 (A), D72.1 (A), D78.1 (A), D84.1 (A), D90.1 (A)
- net at SW2.2: now also D2.1 (A); no longer D2.2 (K)
- net at SW4.2: now also D4.1 (A); no longer D4.2 (K)
- net at SW3.2: now also D3.1 (A); no longer D3.2 (K)
- net at SW6.2: now also D6.1 (A); no longer D6.2 (K)
- net at SW5.2: now also D5.1 (A); no longer D5.2 (K)
- net at SW8.2: now also D8.1 (A); no longer D8.2 (K)
- net at SW7.2: now also D7.1 (A); no longer D7.2 (K)
- net at SW10.2: now also D10.1 (A); no longer D10.2 (K)
- net at SW9.2: now also D9.1 (A); no longer D9.2 (K)
- net at SW12.2: now also D12.1 (A); no longer D12.2 (K)
- net at SW11.2: now also D11.1 (A); no longer D11.2 (K)
- net at SW14.2: now also D14.1 (A); no longer D14.2 (K)
- net at SW13.2: now also D13.1 (A); no longer D13.2 (K)
- net at SW16.2: now also D16.1 (A); no longer D16.2 (K)
- net at SW15.2: now also D15.1 (A); no longer D15.2 (K)
- net at SW18.2: now also D18.1 (A); no longer D18.2 (K)
- net at SW17.2: now also D17.1 (A); no longer D17.2 (K)
- net at SW20.2: now also D20.1 (A); no longer D20.2 (K)
- net at SW19.2: now also D19.1 (A); no longer D19.2 (K)
- net at SW22.2: now also D22.1 (A); no longer D22.2 (K)
- net at SW21.2: now also D21.1 (A); no longer D21.2 (K)
- net at SW24.2: now also D24.1 (A); no longer D24.2 (K)
- net at SW23.2: now also D23.1 (A); no longer D23.2 (K)
- net at SW26.2: now also D26.1 (A); no longer D26.2 (K)
- net at SW25.2: now also D25.1 (A); no longer D25.2 (K)
- net at SW28.2: now also D28.1 (A); no longer D28.2 (K)
- net at SW27.2: now also D27.1 (A); no longer D27.2 (K)
- net at SW30.2: now also D30.1 (A); no longer D30.2 (K)
- net at SW29.2: now also D29.1 (A); no longer D29.2 (K)
- net at SW32.2: now also D32.1 (A); no longer D32.2 (K)
- net at SW31.2: now also D31.1 (A); no longer D31.2 (K)
- net at SW34.2: now also D34.1 (A); no longer D34.2 (K)
- net at SW33.2: now also D33.1 (A); no longer D33.2 (K)
- net at SW36.2: now also D36.1 (A); no longer D36.2 (K)
- net at SW35.2: now also D35.1 (A); no longer D35.2 (K)
- net at SW38.2: now also D38.1 (A); no longer D38.2 (K)
- net at SW37.2: now also D37.1 (A); no longer D37.2 (K)
- net at SW40.2: now also D40.1 (A); no longer D40.2 (K)
- net at SW39.2: now also D39.1 (A); no longer D39.2 (K)
- net at SW42.2: now also D42.1 (A); no longer D42.2 (K)
- net at SW41.2: now also D41.1 (A); no longer D41.2 (K)
- net at SW44.2: now also D44.1 (A); no longer D44.2 (K)
- net at SW43.2: now also D43.1 (A); no longer D43.2 (K)
- net at SW46.2: now also D46.1 (A); no longer D46.2 (K)
- net at SW45.2: now also D45.1 (A); no longer D45.2 (K)
- net at SW48.2: now also D48.1 (A); no longer D48.2 (K)
- net at SW47.2: now also D47.1 (A); no longer D47.2 (K)
- net at SW50.2: now also D50.1 (A); no longer D50.2 (K)
- net at SW49.2: now also D49.1 (A); no longer D49.2 (K)
- net at SW52.2: now also D52.1 (A); no longer D52.2 (K)
- net at SW51.2: now also D51.1 (A); no longer D51.2 (K)
- net at SW54.2: now also D54.1 (A); no longer D54.2 (K)
- net at SW53.2: now also D53.1 (A); no longer D53.2 (K)
- net at SW56.2: now also D56.1 (A); no longer D56.2 (K)
- net at SW55.2: now also D55.1 (A); no longer D55.2 (K)
- net at SW58.2: now also D58.1 (A); no longer D58.2 (K)
- net at SW57.2: now also D57.1 (A); no longer D57.2 (K)
- net at SW60.2: now also D60.1 (A); no longer D60.2 (K)
- net at SW59.2: now also D59.1 (A); no longer D59.2 (K)
- net at SW62.2: now also D62.1 (A); no longer D62.2 (K)
- net at SW61.2: now also D61.1 (A); no longer D61.2 (K)
- net at SW64.2: now also D64.1 (A); no longer D64.2 (K)
- net at SW63.2: now also D63.1 (A); no longer D63.2 (K)
- net at SW66.2: now also D66.1 (A); no longer D66.2 (K)
- net at SW68.2: now also D68.1 (A); no longer D68.2 (K)
- net at SW67.2: now also D67.1 (A); no longer D67.2 (K)
- net at SW70.2: now also D70.1 (A); no longer D70.2 (K)
- net at SW69.2: now also D69.1 (A); no longer D69.2 (K)
- net at SW72.2: now also D72.1 (A); no longer D72.2 (K)
- net at SW71.2: now also D71.1 (A); no longer D71.2 (K)
- net at SW74.2: now also D74.1 (A); no longer D74.2 (K)
- net at SW73.2: now also D73.1 (A); no longer D73.2 (K)
- net at SW76.2: now also D76.1 (A); no longer D76.2 (K)
- net at SW75.2: now also D75.1 (A); no longer D75.2 (K)
- net at SW78.2: now also D78.1 (A); no longer D78.2 (K)
- net at SW77.2: now also D77.1 (A); no longer D77.2 (K)
- net at SW80.2: now also D80.1 (A); no longer D80.2 (K)
- net at SW79.2: now also D79.1 (A); no longer D79.2 (K)
- net at SW82.2: now also D82.1 (A); no longer D82.2 (K)
- net at SW81.2: now also D81.1 (A); no longer D81.2 (K)
- net at SW84.2: now also D84.1 (A); no longer D84.2 (K)
- net at SW83.2: now also D83.1 (A); no longer D83.2 (K)
- net at SW86.2: now also D86.1 (A); no longer D86.2 (K)
- net at SW85.2: now also D85.1 (A); no longer D85.2 (K)
- net at SW88.2: now also D88.1 (A); no longer D88.2 (K)
- net at SW87.2: now also D87.1 (A); no longer D87.2 (K)
- net at SW90.2: now also D90.1 (A); no longer D90.2 (K)
- net at SW89.2: now also D89.1 (A); no longer D89.2 (K)
- new net QHSER': U5.9 (QH'), U6.14 (SER)

Commit message: 再度配線しなおした
Parts:
- D1, D10, D11, D12, D13, D14, D15, D16, D17, D18, D19, D2, D20, D21, D22, D23, D24, D25, D26, D27, D28, D29, D3, D30, D31, D32, D33, D34, D35, D36, D37, D38, D39, D4, D40, D41, D42, D43, D44, D45, D46, D47, D48, D49, D5, D50, D51, D52, D53, D54, D55, D56, D57, D58, D59, D6, D60, D61, D62, D63, D64, D65, D66, D67, D68, D69, D7, D70, D71, D72, D73, D74, D75, D76, D77, D78, D79, D8, D80, D81, D82, D83, D84, D85, D86, D87, D88, D89, D9, D90: symbol Simulation_SPICE:DIODE -> Device:D
- U1, U2: footprint kbd:ProMicro_v3.5 -> kbd:ProMicro_v3.6
- U3, U4, U5, U6: footprint Housings_DIP:DIP-16_W7.62mm_Socket -> kbd:SN74HC595_DIP-16_W7.62mm_Socket_2
Connections:
- net row00: now also D13.1 (K), D19.1 (K), D25.1 (K), D31.1 (K), D37.1 (K), D43.1 (K), D49.1 (K), D55.1 (K), D61.1 (K), D67.1 (K), D7.1 (K), D73.1 (K), D79.1 (K), D85.1 (K); no longer D13.2 (K), D19.2 (K), D25.2 (K), D31.2 (K), D37.2 (K), D43.2 (K), D49.2 (K), D55.2 (K), D61.2 (K), D67.2 (K), D7.2 (K), D73.2 (K), D79.2 (K), D85.2 (K)
- net row01: now also D14.1 (K), D2.1 (K), D20.1 (K), D26.1 (K), D32.1 (K), D38.1 (K), D44.1 (K), D50.1 (K), D56.1 (K), D62.1 (K), D68.1 (K), D74.1 (K), D8.1 (K), D80.1 (K), D86.1 (K); no longer D14.2 (K), D2.2 (K), D20.2 (K), D26.2 (K), D32.2 (K), D38.2 (K), D44.2 (K), D50.2 (K), D56.2 (K), D62.2 (K), D68.2 (K), D74.2 (K), D8.2 (K), D80.2 (K), D86.2 (K)
- net row02: now also D15.1 (K), D21.1 (K), D27.1 (K), D3.1 (K), D33.1 (K), D39.1 (K), D45.1 (K), D51.1 (K), D57.1 (K), D63.1 (K), D69.1 (K), D75.1 (K), D81.1 (K), D87.1 (K), D9.1 (K); no longer D15.2 (K), D21.2 (K), D27.2 (K), D3.2 (K), D33.2 (K), D39.2 (K), D45.2 (K), D51.2 (K), D57.2 (K), D63.2 (K), D69.2 (K), D75.2 (K), D81.2 (K), D87.2 (K), D9.2 (K)
- net row03: now also D10.1 (K), D16.1 (K), D22.1 (K), D28.1 (K), D34.1 (K), D4.1 (K), D40.1 (K), D46.1 (K), D52.1 (K), D58.1 (K), D64.1 (K), D70.1 (K), D76.1 (K), D82.1 (K), D88.1 (K); no longer D10.2 (K), D16.2 (K), D22.2 (K), D28.2 (K), D34.2 (K), D4.2 (K), D40.2 (K), D46.2 (K), D52.2 (K), D58.2 (K), D64.2 (K), D70.2 (K), D76.2 (K), D82.2 (K), D88.2 (K)
- net row04: now also D11.1 (K), D17.1 (K), D23.1 (K), D29.1 (K), D35.1 (K), D41.1 (K), D47.1 (K), D5.1 (K), D53.1 (K), D59.1 (K), D71.1 (K), D77.1 (K), D83.1 (K), D89.1 (K); no longer D11.2 (K), D17.2 (K), D23.2 (K), D29.2 (K), D35.2 (K), D41.2 (K), D47.2 (K), D5.2 (K), D53.2 (K), D59.2 (K), D71.2 (K), D77.2 (K), D83.2 (K), D89.2 (K)
- net row05: now also D12.1 (K), D18.1 (K), D24.1 (K), D30.1 (K), D36.1 (K), D42.1 (K), D48.1 (K), D54.1 (K), D6.1 (K), D60.1 (K), D66.1 (K), D72.1 (K), D78.1 (K), D84.1 (K), D90.1 (K); no longer D12.2 (K), D18.2 (K), D24.2 (K), D30.2 (K), D36.2 (K), D42.2 (K), D48.2 (K), D54.2 (K), D6.2 (K), D60.2 (K), D66.2 (K), D72.2 (K), D78.2 (K), D84.2 (K), D90.2 (K)
- net at SW2.2: now also D2.2 (A); no longer D2.1 (A)
- net at SW4.2: now also D4.2 (A); no longer D4.1 (A)
- net at SW3.2: now also D3.2 (A); no longer D3.1 (A)
- net at SW6.2: now also D6.2 (A); no longer D6.1 (A)
- net at SW5.2: now also D5.2 (A); no longer D5.1 (A)
- net at SW8.2: now also D8.2 (A); no longer D8.1 (A)
- net at SW7.2: now also D7.2 (A); no longer D7.1 (A)
- net at SW10.2: now also D10.2 (A); no longer D10.1 (A)
- net at SW9.2: now also D9.2 (A); no longer D9.1 (A)
- net at SW12.2: now also D12.2 (A); no longer D12.1 (A)
- net at SW11.2: now also D11.2 (A); no longer D11.1 (A)
- net at SW14.2: now also D14.2 (A); no longer D14.1 (A)
- net at SW13.2: now also D13.2 (A); no longer D13.1 (A)
- net at SW16.2: now also D16.2 (A); no longer D16.1 (A)
- net at SW15.2: now also D15.2 (A); no longer D15.1 (A)
- net at SW18.2: now also D18.2 (A); no longer D18.1 (A)
- net at SW17.2: now also D17.2 (A); no longer D17.1 (A)
- net at SW20.2: now also D20.2 (A); no longer D20.1 (A)
- net at SW19.2: now also D19.2 (A); no longer D19.1 (A)
- net at SW22.2: now also D22.2 (A); no longer D22.1 (A)
- net at SW21.2: now also D21.2 (A); no longer D21.1 (A)
- net at SW24.2: now also D24.2 (A); no longer D24.1 (A)
- net at SW23.2: now also D23.2 (A); no longer D23.1 (A)
- net at SW26.2: now also D26.2 (A); no longer D26.1 (A)
- net at SW25.2: now also D25.2 (A); no longer D25.1 (A)
- net at SW28.2: now also D28.2 (A); no longer D28.1 (A)
- net at SW27.2: now also D27.2 (A); no longer D27.1 (A)
- net at SW30.2: now also D30.2 (A); no longer D30.1 (A)
- net at SW29.2: now also D29.2 (A); no longer D29.1 (A)
- net at SW32.2: now also D32.2 (A); no longer D32.1 (A)
- net at SW31.2: now also D31.2 (A); no longer D31.1 (A)
- net at SW34.2: now also D34.2 (A); no longer D34.1 (A)
- net at SW33.2: now also D33.2 (A); no longer D33.1 (A)
- net at SW36.2: now also D36.2 (A); no longer D36.1 (A)
- net at SW35.2: now also D35.2 (A); no longer D35.1 (A)
- net at SW38.2: now also D38.2 (A); no longer D38.1 (A)
- net at SW37.2: now also D37.2 (A); no longer D37.1 (A)
- net at SW40.2: now also D40.2 (A); no longer D40.1 (A)
- net at SW39.2: now also D39.2 (A); no longer D39.1 (A)
- net at SW42.2: now also D42.2 (A); no longer D42.1 (A)
- net at SW41.2: now also D41.2 (A); no longer D41.1 (A)
- net at SW44.2: now also D44.2 (A); no longer D44.1 (A)
- net at SW43.2: now also D43.2 (A); no longer D43.1 (A)
- net at SW46.2: now also D46.2 (A); no longer D46.1 (A)
- net at SW45.2: now also D45.2 (A); no longer D45.1 (A)
- net at SW48.2: now also D48.2 (A); no longer D48.1 (A)
- net at SW47.2: now also D47.2 (A); no longer D47.1 (A)
- net at SW50.2: now also D50.2 (A); no longer D50.1 (A)
- net at SW49.2: now also D49.2 (A); no longer D49.1 (A)
- net at SW52.2: now also D52.2 (A); no longer D52.1 (A)
- net at SW51.2: now also D51.2 (A); no longer D51.1 (A)
- net at SW54.2: now also D54.2 (A); no longer D54.1 (A)
- net at SW53.2: now also D53.2 (A); no longer D53.1 (A)
- net at SW56.2: now also D56.2 (A); no longer D56.1 (A)
- net at SW55.2: now also D55.2 (A); no longer D55.1 (A)
- net at SW58.2: now also D58.2 (A); no longer D58.1 (A)
- net at SW57.2: now also D57.2 (A); no longer D57.1 (A)
- net at SW60.2: now also D60.2 (A); no longer D60.1 (A)
- net at SW59.2: now also D59.2 (A); no longer D59.1 (A)
- net at SW62.2: now also D62.2 (A); no longer D62.1 (A)
- net at SW61.2: now also D61.2 (A); no longer D61.1 (A)
- net at SW64.2: now also D64.2 (A); no longer D64.1 (A)
- net at SW63.2: now also D63.2 (A); no longer D63.1 (A)
- net at SW66.2: now also D66.2 (A); no longer D66.1 (A)
- net at SW68.2: now also D68.2 (A); no longer D68.1 (A)
- net at SW67.2: now also D67.2 (A); no longer D67.1 (A)
- net at SW70.2: now also D70.2 (A); no longer D70.1 (A)
- net at SW69.2: now also D69.2 (A); no longer D69.1 (A)
- net at SW72.2: now also D72.2 (A); no longer D72.1 (A)
- net at SW71.2: now also D71.2 (A); no longer D71.1 (A)
- net at SW74.2: now also D74.2 (A); no longer D74.1 (A)
- net at SW73.2: now also D73.2 (A); no longer D73.1 (A)
- net at SW76.2: now also D76.2 (A); no longer D76.1 (A)
- net at SW75.2: now also D75.2 (A); no longer D75.1 (A)
- net at SW78.2: now also D78.2 (A); no longer D78.1 (A)
- net at SW77.2: now also D77.2 (A); no longer D77.1 (A)
- net at SW80.2: now also D80.2 (A); no longer D80.1 (A)
- net at SW79.2: now also D79.2 (A); no longer D79.1 (A)
- net at SW82.2: now also D82.2 (A); no longer D82.1 (A)
- net at SW81.2: now also D81.2 (A); no longer D81.1 (A)
- net at SW84.2: now also D84.2 (A); no longer D84.1 (A)
- net at SW83.2: now also D83.2 (A); no longer D83.1 (A)
- net at SW86.2: now also D86.2 (A); no longer D86.1 (A)
- net at SW85.2: now also D85.2 (A); no longer D85.1 (A)
- net at SW88.2: now also D88.2 (A); no longer D88.1 (A)
- net at SW87.2: now also D87.2 (A); no longer D87.1 (A)
- net at SW90.2: now also D90.2 (A); no longer D90.1 (A)
- net at SW89.2: now also D89.2 (A); no longer D89.1 (A)
- no-connect marks 59 -> 58
Other:
- moved on the sheet: D1, D10, D11, D12, D13, D14, D15, D16, D17, D18, D19, D2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
