File: fan/fan.kicad_pcb (KiCad board)
At the start: 2 copper layers, 297.2 x 263.7 mm, 196 parts, among them J2 Pi, SW1 SW_PUSH, SW10 SW_PUSH, SW11 SW_PUSH, SW12 SW_PUSH, SW13 SW_PUSH, SW14 SW_PUSH, SW15 SW_PUSH, SW16 SW_PUSH, SW17 SW_PUSH, SW18 SW_PUSH, SW19 SW_PUSH, SW2 SW_PUSH, SW20 SW_PUSH, SW21 SW_PUSH, SW22 SW_PUSH, SW23 SW_PUSH, SW24 SW_PUSH, SW25 SW_PUSH, SW26 SW_PUSH, SW27 SW_PUSH, SW28 SW_PUSH, SW29 SW_PUSH, SW3 SW_PUSH, SW30 SW_PUSH, SW31 SW_PUSH, SW32 SW_PUSH, SW33 SW_PUSH, SW34 SW_PUSH, SW35 SW_PUSH, SW36 SW_PUSH, SW37 SW_PUSH, SW38 SW_PUSH, SW39 SW_PUSH, SW4 SW_PUSH, SW40 SW_PUSH, SW41 SW_PUSH, SW42 SW_PUSH, SW43 SW_PUSH, SW44 SW_PUSH, SW45 SW_PUSH, SW46 SW_PUSH, SW47 SW_PUSH, SW48 SW_PUSH, SW49 SW_PUSH, SW5 SW_PUSH, SW50 SW_PUSH, SW51 SW_PUSH, SW52 SW_PUSH, SW53 SW_PUSH, SW54 SW_PUSH, SW55 SW_PUSH, SW56 SW_PUSH, SW57 SW_PUSH, SW58 SW_PUSH, SW59 SW_PUSH, SW6 SW_PUSH, SW60 SW_PUSH, SW61 SW_PUSH, SW62 SW_PUSH, SW63 SW_PUSH, SW64 SW_PUSH, SW65 SW_PUSH, SW66 SW_PUSH, SW67 SW_PUSH, SW68 SW_PUSH, SW69 SW_PUSH, SW7 SW_PUSH, SW70 SW_PUSH, SW71 SW_PUSH, SW72 SW_PUSH, SW73 SW_PUSH, SW74 SW_PUSH, SW75 SW_PUSH, SW76 SW_PUSH, SW77 SW_PUSH, SW78 SW_PUSH, SW79 SW_PUSH, SW8 SW_PUSH, SW80 SW_PUSH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

Commit message: 大幅に手戻り 配線最初から
Parts:
- moved U5 0.09 mm to (214.2, 119.4)
- moved U6 0.08 mm to (234.8, 121.6)
Connections:
- D10 pad 1: row03 -> Net-(D10-Pad1)
- D10 pad 2: Net-(D10-Pad2) -> row03
- D11 pad 1: row04 -> Net-(D11-Pad1)
- D11 pad 2: Net-(D11-Pad2) -> row04
- D12 pad 1: row05 -> Net-(D12-Pad1)
- D12 pad 2: Net-(D12-Pad2) -> row05
- D13 pad 1: row00 -> Net-(D13-Pad1)
- D13 pad 2: Net-(D13-Pad2) -> row00
- D14 pad 1: row01 -> Net-(D14-Pad1)
- D14 pad 2: Net-(D14-Pad2) -> row01
- D15 pad 1: row02 -> Net-(D15-Pad1)
- D15 pad 2: Net-(D15-Pad2) -> row02
- D16 pad 1: row03 -> Net-(D16-Pad1)
- D16 pad 2: Net-(D16-Pad2) -> row03
- D17 pad 1: row04 -> Net-(D17-Pad1)
- D17 pad 2: Net-(D17-Pad2) -> row04
- D18 pad 1: row05 -> Net-(D18-Pad1)
- D18 pad 2: Net-(D18-Pad2) -> row05
- D19 pad 1: row00 -> Net-(D19-Pad1)
- D19 pad 2: Net-(D19-Pad2) -> row00
- D2 pad 1: row01 -> Net-(D2-Pad1)
- D2 pad 2: Net-(D2-Pad2) -> row01
- D20 pad 1: row01 -> Net-(D20-Pad1)
- D20 pad 2: Net-(D20-Pad2) -> row01
- D21 pad 1: row02 -> Net-(D21-Pad1)
- D21 pad 2: Net-(D21-Pad2) -> row02
- D22 pad 1: row03 -> Net-(D22-Pad1)
- D22 pad 2: Net-(D22-Pad2) -> row03
- D23 pad 1: row04 -> Net-(D23-Pad1)
- D23 pad 2: Net-(D23-Pad2) -> row04
- D24 pad 1: row05 -> Net-(D24-Pad1)
- D24 pad 2: Net-(D24-Pad2) -> row05
- D25 pad 1: row00 -> Net-(D25-Pad1)
- D25 pad 2: Net-(D25-Pad2) -> row00
- D26 pad 1: row01 -> Net-(D26-Pad1)
- D26 pad 2: Net-(D26-Pad2) -> row01
- D27 pad 1: row02 -> Net-(D27-Pad1)
- D27 pad 2: Net-(D27-Pad2) -> row02
- D28 pad 1: row03 -> Net-(D28-Pad1)
- D28 pad 2: Net-(D28-Pad2) -> row03
- D29 pad 1: row04 -> Net-(D29-Pad1)
- D29 pad 2: Net-(D29-Pad2) -> row04
- D3 pad 1: row02 -> Net-(D3-Pad1)
- D3 pad 2: Net-(D3-Pad2) -> row02
- D30 pad 1: row05 -> Net-(D30-Pad1)
- D30 pad 2: Net-(D30-Pad2) -> row05
- D31 pad 1: row00 -> Net-(D31-Pad1)
- D31 pad 2: Net-(D31-Pad2) -> row00
- D32 pad 1: row01 -> Net-(D32-Pad1)
- D32 pad 2: Net-(D32-Pad2) -> row01
- D33 pad 1: row02 -> Net-(D33-Pad1)
- D33 pad 2: Net-(D33-Pad2) -> row02
- D34 pad 1: row03 -> Net-(D34-Pad1)
- D34 pad 2: Net-(D34-Pad2) -> row03
- D35 pad 1: row04 -> Net-(D35-Pad1)
- D35 pad 2: Net-(D35-Pad2) -> row04
- D36 pad 1: row05 -> Net-(D36-Pad1)
- D36 pad 2: Net-(D36-Pad2) -> row05
- D37 pad 1: row00 -> Net-(D37-Pad1)
- D37 pad 2: Net-(D37-Pad2) -> row00
- D38 pad 1: row01 -> Net-(D38-Pad1)
- D38 pad 2: Net-(D38-Pad2) -> row01
- D39 pad 1: row02 -> Net-(D39-Pad1)
- D39 pad 2: Net-(D39-Pad2) -> row02
- D4 pad 1: row03 -> Net-(D4-Pad1)
- D4 pad 2: Net-(D4-Pad2) -> row03
- D40 pad 1: row03 -> Net-(D40-Pad1)
- D40 pad 2: Net-(D40-Pad2) -> row03
- D41 pad 1: row04 -> Net-(D41-Pad1)
- D41 pad 2: Net-(D41-Pad2) -> row04
- D42 pad 1: row05 -> Net-(D42-Pad1)
- D42 pad 2: Net-(D42-Pad2) -> row05
- D43 pad 1: row00 -> Net-(D43-Pad1)
- D43 pad 2: Net-(D43-Pad2) -> row00
- D44 pad 1: row01 -> Net-(D44-Pad1)
- D44 pad 2: Net-(D44-Pad2) -> row01
- D45 pad 1: row02 -> Net-(D45-Pad1)
- D45 pad 2: Net-(D45-Pad2) -> row02
- D46 pad 1: row03 -> Net-(D46-Pad1)
- D46 pad 2: Net-(D46-Pad2) -> row03
- D47 pad 1: row04 -> Net-(D47-Pad1)
- D47 pad 2: Net-(D47-Pad2) -> row04
- D48 pad 1: row05 -> Net-(D48-Pad1)
- D48 pad 2: Net-(D48-Pad2) -> row05
- D49 pad 1: row00 -> Net-(D49-Pad1)
- D49 pad 2: Net-(D49-Pad2) -> row00
- D5 pad 1: row04 -> Net-(D5-Pad1)
- D5 pad 2: Net-(D5-Pad2) -> row04
- D50 pad 1: row01 -> Net-(D50-Pad1)
- D50 pad 2: Net-(D50-Pad2) -> row01
- D51 pad 1: row02 -> Net-(D51-Pad1)
- D51 pad 2: Net-(D51-Pad2) -> row02
- D52 pad 1: row03 -> Net-(D52-Pad1)
- D52 pad 2: Net-(D52-Pad2) -> row03
- D53 pad 1: row04 -> Net-(D53-Pad1)
- D53 pad 2: Net-(D53-Pad2) -> row04
- D54 pad 1: row05 -> Net-(D54-Pad1)
- D54 pad 2: Net-(D54-Pad2) -> row05
- D55 pad 1: row00 -> Net-(D55-Pad1)
- D55 pad 2: Net-(D55-Pad2) -> row00
- D56 pad 1: row01 -> Net-(D56-Pad1)
- D56 pad 2: Net-(D56-Pad2) -> row01
- D57 pad 1: row02 -> Net-(D57-Pad1)
- D57 pad 2: Net-(D57-Pad2) -> row02
- D58 pad 1: row03 -> Net-(D58-Pad1)
- D58 pad 2: Net-(D58-Pad2) -> row03
- D59 pad 1: row04 -> Net-(D59-Pad1)
- D59 pad 2: Net-(D59-Pad2) -> row04
- D6 pad 1: row05 -> Net-(D6-Pad1)
- D6 pad 2: Net-(D6-Pad2) -> row05
- D60 pad 1: row05 -> Net-(D60-Pad1)
- D60 pad 2: Net-(D60-Pad2) -> row05
- D61 pad 1: row00 -> Net-(D61-Pad1)
- D61 pad 2: Net-(D61-Pad2) -> row00
- D62 pad 1: row01 -> Net-(D62-Pad1)
- D62 pad 2: Net-(D62-Pad2) -> row01
- D63 pad 1: row02 -> Net-(D63-Pad1)
- D63 pad 2: Net-(D63-Pad2) -> row02
- D64 pad 1: row03 -> Net-(D64-Pad1)
- D64 pad 2: Net-(D64-Pad2) -> row03
- D66 pad 1: row05 -> Net-(D66-Pad1)
- D66 pad 2: Net-(D66-Pad2) -> row05
- D67 pad 1: row00 -> Net-(D67-Pad1)
- D67 pad 2: Net-(D67-Pad2) -> row00
- D68 pad 1: row01 -> Net-(D68-Pad1)
- D68 pad 2: Net-(D68-Pad2) -> row01
- D69 pad 1: row02 -> Net-(D69-Pad1)
- D69 pad 2: Net-(D69-Pad2) -> row02
- D7 pad 1: row00 -> Net-(D7-Pad1)
- D7 pad 2: Net-(D7-Pad2) -> row00
- D70 pad 1: row03 -> Net-(D70-Pad1)
- D70 pad 2: Net-(D70-Pad2) -> row03
- D71 pad 1: row04 -> Net-(D71-Pad1)
- D71 pad 2: Net-(D71-Pad2) -> row04
- D72 pad 1: row05 -> Net-(D72-Pad1)
- D72 pad 2: Net-(D72-Pad2) -> row05
- D73 pad 1: row00 -> Net-(D73-Pad1)
- D73 pad 2: Net-(D73-Pad2) -> row00
- D74 pad 1: row01 -> Net-(D74-Pad1)
- D74 pad 2: Net-(D74-Pad2) -> row01
- D75 pad 1: row02 -> Net-(D75-Pad1)
- D75 pad 2: Net-(D75-Pad2) -> row02
- D76 pad 1: row03 -> Net-(D76-Pad1)
- D76 pad 2: Net-(D76-Pad2) -> row03
- D77 pad 1: row04 -> Net-(D77-Pad1)
- D77 pad 2: Net-(D77-Pad2) -> row04
- D78 pad 1: row05 -> Net-(D78-Pad1)
- D78 pad 2: Net-(D78-Pad2) -> row05
- D79 pad 1: row00 -> Net-(D79-Pad1)
- D79 pad 2: Net-(D79-Pad2) -> row00
- D8 pad 1: row01 -> Net-(D8-Pad1)
- D8 pad 2: Net-(D8-Pad2) -> row01
- D80 pad 1: row01 -> Net-(D80-Pad1)
- D80 pad 2: Net-(D80-Pad2) -> row01
- D81 pad 1: row02 -> Net-(D81-Pad1)
- D81 pad 2: Net-(D81-Pad2) -> row02
- D82 pad 1: row03 -> Net-(D82-Pad1)
- D82 pad 2: Net-(D82-Pad2) -> row03
- D83 pad 1: row04 -> Net-(D83-Pad1)
- D83 pad 2: Net-(D83-Pad2) -> row04
- D84 pad 1: row05 -> Net-(D84-Pad1)
- D84 pad 2: Net-(D84-Pad2) -> row05
- D85 pad 1: row00 -> Net-(D85-Pad1)
- D85 pad 2: Net-(D85-Pad2) -> row00
- D86 pad 1: row01 -> Net-(D86-Pad1)
- D86 pad 2: Net-(D86-Pad2) -> row01
- D87 pad 1: row02 -> Net-(D87-Pad1)
- D87 pad 2: Net-(D87-Pad2) -> row02
- D88 pad 1: row03 -> Net-(D88-Pad1)
- D88 pad 2: Net-(D88-Pad2) -> row03
- D89 pad 1: row04 -> Net-(D89-Pad1)
- D89 pad 2: Net-(D89-Pad2) -> row04
- D9 pad 1: row02 -> Net-(D9-Pad1)
- D9 pad 2: Net-(D9-Pad2) -> row02
- D90 pad 1: row05 -> Net-(D90-Pad1)
- D90 pad 2: Net-(D90-Pad2) -> row05
- SW10 pad 2: Net-(D10-Pad2) -> Net-(D10-Pad1)
- SW11 pad 2: Net-(D11-Pad2) -> Net-(D11-Pad1)
- SW12 pad 2: Net-(D12-Pad2) -> Net-(D12-Pad1)
- SW13 pad 2: Net-(D13-Pad2) -> Net-(D13-Pad1)
- SW14 pad 2: Net-(D14-Pad2) -> Net-(D14-Pad1)
- SW15 pad 2: Net-(D15-Pad2) -> Net-(D15-Pad1)
- SW16 pad 2: Net-(D16-Pad2) -> Net-(D16-Pad1)
- SW17 pad 2: Net-(D17-Pad2) -> Net-(D17-Pad1)
- SW18 pad 2: Net-(D18-Pad2) -> Net-(D18-Pad1)
- SW19 pad 2: Net-(D19-Pad2) -> Net-(D19-Pad1)
- SW2 pad 2: Net-(D2-Pad2) -> Net-(D2-Pad1)
- SW20 pad 2: Net-(D20-Pad2) -> Net-(D20-Pad1)
- SW21 pad 2: Net-(D21-Pad2) -> Net-(D21-Pad1)
- SW22 pad 2: Net-(D22-Pad2) -> Net-(D22-Pad1)
- SW23 pad 2: Net-(D23-Pad2) -> Net-(D23-Pad1)
- SW24 pad 2: Net-(D24-Pad2) -> Net-(D24-Pad1)
- SW25 pad 2: Net-(D25-Pad2) -> Net-(D25-Pad1)
- SW26 pad 2: Net-(D26-Pad2) -> Net-(D26-Pad1)
- SW27 pad 2: Net-(D27-Pad2) -> Net-(D27-Pad1)
- SW28 pad 2: Net-(D28-Pad2) -> Net-(D28-Pad1)
- SW29 pad 2: Net-(D29-Pad2) -> Net-(D29-Pad1)
- SW3 pad 2: Net-(D3-Pad2) -> Net-(D3-Pad1)
- SW30 pad 2: Net-(D30-Pad2) -> Net-(D30-Pad1)
- SW31 pad 2: Net-(D31-Pad2) -> Net-(D31-Pad1)
- SW32 pad 2: Net-(D32-Pad2) -> Net-(D32-Pad1)
- SW33 pad 2: Net-(D33-Pad2) -> Net-(D33-Pad1)
- SW34 pad 2: Net-(D34-Pad2) -> Net-(D34-Pad1)
- SW35 pad 2: Net-(D35-Pad2) -> Net-(D35-Pad1)
- SW36 pad 2: Net-(D36-Pad2) -> Net-(D36-Pad1)
- SW37 pad 2: Net-(D37-Pad2) -> Net-(D37-Pad1)
- SW38 pad 2: Net-(D38-Pad2) -> Net-(D38-Pad1)
- SW39 pad 2: Net-(D39-Pad2) -> Net-(D39-Pad1)
- SW4 pad 2: Net-(D4-Pad2) -> Net-(D4-Pad1)
- SW40 pad 2: Net-(D40-Pad2) -> Net-(D40-Pad1)
- SW41 pad 2: Net-(D41-Pad2) -> Net-(D41-Pad1)
- SW42 pad 2: Net-(D42-Pad2) -> Net-(D42-Pad1)
- SW43 pad 2: Net-(D43-Pad2) -> Net-(D43-Pad1)
- SW44 pad 2: Net-(D44-Pad2) -> Net-(D44-Pad1)
- SW45 pad 2: Net-(D45-Pad2) -> Net-(D45-Pad1)
- SW46 pad 2: Net-(D46-Pad2) -> Net-(D46-Pad1)
- SW47 pad 2: Net-(D47-Pad2) -> Net-(D47-Pad1)
- SW48 pad 2: Net-(D48-Pad2) -> Net-(D48-Pad1)
- SW49 pad 2: Net-(D49-Pad2) -> Net-(D49-Pad1)
- SW5 pad 2: Net-(D5-Pad2) -> Net-(D5-Pad1)
- SW50 pad 2: Net-(D50-Pad2) -> Net-(D50-Pad1)
- SW51 pad 2: Net-(D51-Pad2) -> Net-(D51-Pad1)
- SW52 pad 2: Net-(D52-Pad2) -> Net-(D52-Pad1)
- SW53 pad 2: Net-(D53-Pad2) -> Net-(D53-Pad1)
- SW54 pad 2: Net-(D54-Pad2) -> Net-(D54-Pad1)
- SW55 pad 2: Net-(D55-Pad2) -> Net-(D55-Pad1)
- SW56 pad 2: Net-(D56-Pad2) -> Net-(D56-Pad1)
- SW57 pad 2: Net-(D57-Pad2) -> Net-(D57-Pad1)
- SW58 pad 2: Net-(D58-Pad2) -> Net-(D58-Pad1)
- SW59 pad 2: Net-(D59-Pad2) -> Net-(D59-Pad1)
- SW6 pad 2: Net-(D6-Pad2) -> Net-(D6-Pad1)
- SW60 pad 2: Net-(D60-Pad2) -> Net-(D60-Pad1)
- SW61 pad 2: Net-(D61-Pad2) -> Net-(D61-Pad1)
- SW62 pad 2: Net-(D62-Pad2) -> Net-(D62-Pad1)
- SW63 pad 2: Net-(D63-Pad2) -> Net-(D63-Pad1)
- SW64 pad 2: Net-(D64-Pad2) -> Net-(D64-Pad1)
- SW66 pad 2: Net-(D66-Pad2) -> Net-(D66-Pad1)
- SW67 pad 2: Net-(D67-Pad2) -> Net-(D67-Pad1)
- SW68 pad 2: Net-(D68-Pad2) -> Net-(D68-Pad1)
- SW69 pad 2: Net-(D69-Pad2) -> Net-(D69-Pad1)
- SW7 pad 2: Net-(D7-Pad2) -> Net-(D7-Pad1)
- SW70 pad 2: Net-(D70-Pad2) -> Net-(D70-Pad1)
- SW71 pad 2: Net-(D71-Pad2) -> Net-(D71-Pad1)
- SW72 pad 2: Net-(D72-Pad2) -> Net-(D72-Pad1)
- SW73 pad 2: Net-(D73-Pad2) -> Net-(D73-Pad1)
- SW74 pad 2: Net-(D74-Pad2) -> Net-(D74-Pad1)
- SW75 pad 2: Net-(D75-Pad2) -> Net-(D75-Pad1)
- SW76 pad 2: Net-(D76-Pad2) -> Net-(D76-Pad1)
- SW77 pad 2: Net-(D77-Pad2) -> Net-(D77-Pad1)
- SW78 pad 2: Net-(D78-Pad2) -> Net-(D78-Pad1)
- SW79 pad 2: Net-(D79-Pad2) -> Net-(D79-Pad1)
- SW8 pad 2: Net-(D8-Pad2) -> Net-(D8-Pad1)
- SW80 pad 2: Net-(D80-Pad2) -> Net-(D80-Pad1)
- SW81 pad 2: Net-(D81-Pad2) -> Net-(D81-Pad1)
- SW82 pad 2: Net-(D82-Pad2) -> Net-(D82-Pad1)
- SW83 pad 2: Net-(D83-Pad2) -> Net-(D83-Pad1)
- SW84 pad 2: Net-(D84-Pad2) -> Net-(D84-Pad1)
- SW85 pad 2: Net-(D85-Pad2) -> Net-(D85-Pad1)
- SW86 pad 2: Net-(D86-Pad2) -> Net-(D86-Pad1)
- SW87 pad 2: Net-(D87-Pad2) -> Net-(D87-Pad1)
- SW88 pad 2: Net-(D88-Pad2) -> Net-(D88-Pad1)
- SW89 pad 2: Net-(D89-Pad2) -> Net-(D89-Pad1)
- SW9 pad 2: Net-(D9-Pad2) -> Net-(D9-Pad1)
- SW90 pad 2: Net-(D90-Pad2) -> Net-(D90-Pad1)
- U5 pad 9: QHSER -> QHSER'
- U6 pad 14: QHSER -> QHSER'
Routing:
- net row02: track 609.5 -> 18.4 mm, vias 6 -> 0
- net row03: track 565.6 -> 18.4 mm, vias 4 -> 0
- net row04: track 545.8 -> 18.4 mm, vias 3 -> 0
- net row05: track 512.4 -> 18.4 mm, vias 2 -> 0
- net row01: track 509.8 -> 19.4 mm, vias 3 -> 0
- net col14: track 484.9 -> 11.2 mm, vias 4 -> 0
- net col13: track 476.9 -> 12.3 mm, vias 5 -> 0
- net col12: track 461.0 -> 12.5 mm, vias 7 -> 0
- net col10: track 457.1 -> 12.3 mm, vias 7 -> 0
- net row00: track 454.4 -> 18.4 mm, vias 1 -> 0
- net col11: track 430.3 -> 12.3 mm, vias 6 -> 0
- net col09: track 365.3 -> 12.3 mm, vias 5 -> 0
- net col01: track 329.8 -> 12.3 mm, vias 4 -> 0
- net col00: track 327.9 -> 17.9 mm, vias 4 -> 0
- net col05: track 304.3 -> 12.3 mm, vias 6 -> 0
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
Commit message: 再度配線しなおした
Parts:
- removed Ref** (x2): Val**, kbd:HOLE
- added HOLE2: Val**, kbd:HOLE, F.Cu at (124.1, 273.2)
- added HOLE6: Val**, kbd:HOLE, F.Cu at (262.6, 360.8)
- U1, U2: footprint kbd:ProMicro_v3.5 -> kbd:ProMicro_v3.6
- U3, U4, U5, U6: footprint Housings_DIP:DIP-16_W7.62mm_Socket -> kbd:SN74HC595_DIP-16_W7.62mm_Socket_2
- moved U3 23.5 mm to (233.9, 122.1), turned to 78 degrees
- moved U4 22.9 mm to (254.6, 126.5), turned to 78 degrees
- moved U6 22.0 mm to (256.7, 123.9), turned to 258 degrees
- moved U5 21.8 mm to (236.0, 119.5), turned to 258 degrees
- moved HOLE1 13.9 mm to (126.8, 131.9), turned to 355 degrees
- moved HOLE5 13.4 mm to (384.5, 306.8), turned to 355 degrees
- moved U1 13.3 mm to (201.3, 117.0), turned to 90 degrees
- moved U2 13.0 mm to (202.5, 114.5), turned to 270 degrees
- moved SW91 12.1 mm to (151.5, 135.5), turned to 14 degrees
- moved SW1 12.1 mm to (136.3, 154.2), turned to 15 degrees
- moved SW85 11.8 mm to (364.9, 305.8), turned to 279 degrees
- moved D1 11.7 mm to (145.2, 149.2), turned to 285 degrees
- moved D85 11.6 mm to (368.0, 295.2), turned to 189 degrees
- moved SW2 11.6 mm to (130.4, 176.2), turned to 16 degrees
- moved D2 11.2 mm to (138.5, 168.7), turned to 286 degrees
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- renumbered Ref** to HOLE1, Ref** to HOLE3, Ref** to HOLE4, Ref** to HOLE5
Connections:
- D10 pad 1: Net-(D10-Pad1) -> row03
- D10 pad 2: row03 -> Net-(D10-Pad2)
- D11 pad 1: Net-(D11-Pad1) -> row04
- D11 pad 2: row04 -> Net-(D11-Pad2)
- D12 pad 1: Net-(D12-Pad1) -> row05
- D12 pad 2: row05 -> Net-(D12-Pad2)
- D13 pad 1: Net-(D13-Pad1) -> row00
- D13 pad 2: row00 -> Net-(D13-Pad2)
- D14 pad 1: Net-(D14-Pad1) -> row01
- D14 pad 2: row01 -> Net-(D14-Pad2)
- D15 pad 1: Net-(D15-Pad1) -> row02
- D15 pad 2: row02 -> Net-(D15-Pad2)
- D16 pad 1: Net-(D16-Pad1) -> row03
- D16 pad 2: row03 -> Net-(D16-Pad2)
- D17 pad 1: Net-(D17-Pad1) -> row04
- D17 pad 2: row04 -> Net-(D17-Pad2)
- D18 pad 1: Net-(D18-Pad1) -> row05
- D18 pad 2: row05 -> Net-(D18-Pad2)
- D19 pad 1: Net-(D19-Pad1) -> row00
- D19 pad 2: row00 -> Net-(D19-Pad2)
- D2 pad 1: Net-(D2-Pad1) -> row01
- D2 pad 2: row01 -> Net-(D2-Pad2)
- D20 pad 1: Net-(D20-Pad1) -> row01
- D20 pad 2: row01 -> Net-(D20-Pad2)
- D21 pad 1: Net-(D21-Pad1) -> row02
- D21 pad 2: row02 -> Net-(D21-Pad2)
- D22 pad 1: Net-(D22-Pad1) -> row03
- D22 pad 2: row03 -> Net-(D22-Pad2)
- D23 pad 1: Net-(D23-Pad1) -> row04
- D23 pad 2: row04 -> Net-(D23-Pad2)
- D24 pad 1: Net-(D24-Pad1) -> row05
- D24 pad 2: row05 -> Net-(D24-Pad2)
- D25 pad 1: Net-(D25-Pad1) -> row00
- D25 pad 2: row00 -> Net-(D25-Pad2)
- D26 pad 1: Net-(D26-Pad1) -> row01
- D26 pad 2: row01 -> Net-(D26-Pad2)
- D27 pad 1: Net-(D27-Pad1) -> row02
- D27 pad 2: row02 -> Net-(D27-Pad2)
- D28 pad 1: Net-(D28-Pad1) -> row03
- D28 pad 2: row03 -> Net-(D28-Pad2)
- D29 pad 1: Net-(D29-Pad1) -> row04
- D29 pad 2: row04 -> Net-(D29-Pad2)
- D3 pad 1: Net-(D3-Pad1) -> row02
- D3 pad 2: row02 -> Net-(D3-Pad2)
- D30 pad 1: Net-(D30-Pad1) -> row05
- D30 pad 2: row05 -> Net-(D30-Pad2)
- D31 pad 1: Net-(D31-Pad1) -> row00
- D31 pad 2: row00 -> Net-(D31-Pad2)
- D32 pad 1: Net-(D32-Pad1) -> row01
- D32 pad 2: row01 -> Net-(D32-Pad2)
- D33 pad 1: Net-(D33-Pad1) -> row02
- D33 pad 2: row02 -> Net-(D33-Pad2)
- D34 pad 1: Net-(D34-Pad1) -> row03
- D34 pad 2: row03 -> Net-(D34-Pad2)
- D35 pad 1: Net-(D35-Pad1) -> row04
- D35 pad 2: row04 -> Net-(D35-Pad2)
- D36 pad 1: Net-(D36-Pad1) -> row05
- D36 pad 2: row05 -> Net-(D36-Pad2)
- D37 pad 1: Net-(D37-Pad1) -> row00
- D37 pad 2: row00 -> Net-(D37-Pad2)
- D38 pad 1: Net-(D38-Pad1) -> row01
- D38 pad 2: row01 -> Net-(D38-Pad2)
- D39 pad 1: Net-(D39-Pad1) -> row02
- D39 pad 2: row02 -> Net-(D39-Pad2)
- D4 pad 1: Net-(D4-Pad1) -> row03
- D4 pad 2: row03 -> Net-(D4-Pad2)
- D40 pad 1: Net-(D40-Pad1) -> row03
- D40 pad 2: row03 -> Net-(D40-Pad2)
- D41 pad 1: Net-(D41-Pad1) -> row04
- D41 pad 2: row04 -> Net-(D41-Pad2)
- D42 pad 1: Net-(D42-Pad1) -> row05
- D42 pad 2: row05 -> Net-(D42-Pad2)
- D43 pad 1: Net-(D43-Pad1) -> row00
- D43 pad 2: row00 -> Net-(D43-Pad2)
- D44 pad 1: Net-(D44-Pad1) -> row01
- D44 pad 2: row01 -> Net-(D44-Pad2)
- D45 pad 1: Net-(D45-Pad1) -> row02
- D45 pad 2: row02 -> Net-(D45-Pad2)
- D46 pad 1: Net-(D46-Pad1) -> row03
- D46 pad 2: row03 -> Net-(D46-Pad2)
- D47 pad 1: Net-(D47-Pad1) -> row04
- D47 pad 2: row04 -> Net-(D47-Pad2)
- D48 pad 1: Net-(D48-Pad1) -> row05
- D48 pad 2: row05 -> Net-(D48-Pad2)
- D49 pad 1: Net-(D49-Pad1) -> row00
- D49 pad 2: row00 -> Net-(D49-Pad2)
- D5 pad 1: Net-(D5-Pad1) -> row04
- D5 pad 2: row04 -> Net-(D5-Pad2)
- D50 pad 1: Net-(D50-Pad1) -> row01
- D50 pad 2: row01 -> Net-(D50-Pad2)
- D51 pad 1: Net-(D51-Pad1) -> row02
- D51 pad 2: row02 -> Net-(D51-Pad2)
- D52 pad 1: Net-(D52-Pad1) -> row03
- D52 pad 2: row03 -> Net-(D52-Pad2)
- D53 pad 1: Net-(D53-Pad1) -> row04
- D53 pad 2: row04 -> Net-(D53-Pad2)
- D54 pad 1: Net-(D54-Pad1) -> row05
- D54 pad 2: row05 -> Net-(D54-Pad2)
- D55 pad 1: Net-(D55-Pad1) -> row00
- D55 pad 2: row00 -> Net-(D55-Pad2)
- D56 pad 1: Net-(D56-Pad1) -> row01
- D56 pad 2: row01 -> Net-(D56-Pad2)
- D57 pad 1: Net-(D57-Pad1) -> row02
- D57 pad 2: row02 -> Net-(D57-Pad2)
- D58 pad 1: Net-(D58-Pad1) -> row03
- D58 pad 2: row03 -> Net-(D58-Pad2)
- D59 pad 1: Net-(D59-Pad1) -> row04
- D59 pad 2: row04 -> Net-(D59-Pad2)
- D6 pad 1: Net-(D6-Pad1) -> row05
- D6 pad 2: row05 -> Net-(D6-Pad2)
- D60 pad 1: Net-(D60-Pad1) -> row05
- D60 pad 2: row05 -> Net-(D60-Pad2)
- D61 pad 1: Net-(D61-Pad1) -> row00
- D61 pad 2: row00 -> Net-(D61-Pad2)
- D62 pad 1: Net-(D62-Pad1) -> row01
- D62 pad 2: row01 -> Net-(D62-Pad2)
- D63 pad 1: Net-(D63-Pad1) -> row02
- D63 pad 2: row02 -> Net-(D63-Pad2)
- D64 pad 1: Net-(D64-Pad1) -> row03
- D64 pad 2: row03 -> Net-(D64-Pad2)
- D66 pad 1: Net-(D66-Pad1) -> row05
- D66 pad 2: row05 -> Net-(D66-Pad2)
- D67 pad 1: Net-(D67-Pad1) -> row00
- D67 pad 2: row00 -> Net-(D67-Pad2)
- D68 pad 1: Net-(D68-Pad1) -> row01
- D68 pad 2: row01 -> Net-(D68-Pad2)
- D69 pad 1: Net-(D69-Pad1) -> row02
- D69 pad 2: row02 -> Net-(D69-Pad2)
- D7 pad 1: Net-(D7-Pad1) -> row00
- D7 pad 2: row00 -> Net-(D7-Pad2)
- D70 pad 1: Net-(D70-Pad1) -> row03
- D70 pad 2: row03 -> Net-(D70-Pad2)
- D71 pad 1: Net-(D71-Pad1) -> row04
- D71 pad 2: row04 -> Net-(D71-Pad2)
- D72 pad 1: Net-(D72-Pad1) -> row05
- D72 pad 2: row05 -> Net-(D72-Pad2)
- D73 pad 1: Net-(D73-Pad1) -> row00
- D73 pad 2: row00 -> Net-(D73-Pad2)
- D74 pad 1: Net-(D74-Pad1) -> row01
- D74 pad 2: row01 -> Net-(D74-Pad2)
- D75 pad 1: Net-(D75-Pad1) -> row02
- D75 pad 2: row02 -> Net-(D75-Pad2)
- D76 pad 1: Net-(D76-Pad1) -> row03
- D76 pad 2: row03 -> Net-(D76-Pad2)
- D77 pad 1: Net-(D77-Pad1) -> row04
- D77 pad 2: row04 -> Net-(D77-Pad2)
- D78 pad 1: Net-(D78-Pad1) -> row05
- D78 pad 2: row05 -> Net-(D78-Pad2)
- D79 pad 1: Net-(D79-Pad1) -> row00
- D79 pad 2: row00 -> Net-(D79-Pad2)
- D8 pad 1: Net-(D8-Pad1) -> row01
- D8 pad 2: row01 -> Net-(D8-Pad2)
- D80 pad 1: Net-(D80-Pad1) -> row01
- D80 pad 2: row01 -> Net-(D80-Pad2)
- D81 pad 1: Net-(D81-Pad1) -> row02
- D81 pad 2: row02 -> Net-(D81-Pad2)
- D82 pad 1: Net-(D82-Pad1) -> row03
- D82 pad 2: row03 -> Net-(D82-Pad2)
- D83 pad 1: Net-(D83-Pad1) -> row04
- D83 pad 2: row04 -> Net-(D83-Pad2)
- D84 pad 1: Net-(D84-Pad1) -> row05
- D84 pad 2: row05 -> Net-(D84-Pad2)
- D85 pad 1: Net-(D85-Pad1) -> row00
- D85 pad 2: row00 -> Net-(D85-Pad2)
- D86 pad 1: Net-(D86-Pad1) -> row01
- D86 pad 2: row01 -> Net-(D86-Pad2)
- D87 pad 1: Net-(D87-Pad1) -> row02
- D87 pad 2: row02 -> Net-(D87-Pad2)
- D88 pad 1: Net-(D88-Pad1) -> row03
- D88 pad 2: row03 -> Net-(D88-Pad2)
- D89 pad 1: Net-(D89-Pad1) -> row04
- D89 pad 2: row04 -> Net-(D89-Pad2)
- D9 pad 1: Net-(D9-Pad1) -> row02
- D9 pad 2: row02 -> Net-(D9-Pad2)
- D90 pad 1: Net-(D90-Pad1) -> row05
- D90 pad 2: row05 -> Net-(D90-Pad2)
- SW10 pad 2: Net-(D10-Pad1) -> Net-(D10-Pad2)
- SW11 pad 2: Net-(D11-Pad1) -> Net-(D11-Pad2)
- SW12 pad 2: Net-(D12-Pad1) -> Net-(D12-Pad2)
- SW13 pad 2: Net-(D13-Pad1) -> Net-(D13-Pad2)
- SW14 pad 2: Net-(D14-Pad1) -> Net-(D14-Pad2)
- SW15 pad 2: Net-(D15-Pad1) -> Net-(D15-Pad2)
- SW16 pad 2: Net-(D16-Pad1) -> Net-(D16-Pad2)
- SW17 pad 2: Net-(D17-Pad1) -> Net-(D17-Pad2)
- SW18 pad 2: Net-(D18-Pad1) -> Net-(D18-Pad2)
- SW19 pad 2: Net-(D19-Pad1) -> Net-(D19-Pad2)
- SW2 pad 2: Net-(D2-Pad1) -> Net-(D2-Pad2)
- SW20 pad 2: Net-(D20-Pad1) -> Net-(D20-Pad2)
- SW21 pad 2: Net-(D21-Pad1) -> Net-(D21-Pad2)
- SW22 pad 2: Net-(D22-Pad1) -> Net-(D22-Pad2)
- SW23 pad 2: Net-(D23-Pad1) -> Net-(D23-Pad2)
- SW24 pad 2: Net-(D24-Pad1) -> Net-(D24-Pad2)
- SW25 pad 2: Net-(D25-Pad1) -> Net-(D25-Pad2)
- SW26 pad 2: Net-(D26-Pad1) -> Net-(D26-Pad2)
- SW27 pad 2: Net-(D27-Pad1) -> Net-(D27-Pad2)
- SW28 pad 2: Net-(D28-Pad1) -> Net-(D28-Pad2)
- SW29 pad 2: Net-(D29-Pad1) -> Net-(D29-Pad2)
- SW3 pad 2: Net-(D3-Pad1) -> Net-(D3-Pad2)
- SW30 pad 2: Net-(D30-Pad1) -> Net-(D30-Pad2)
- SW31 pad 2: Net-(D31-Pad1) -> Net-(D31-Pad2)
- SW32 pad 2: Net-(D32-Pad1) -> Net-(D32-Pad2)
- SW33 pad 2: Net-(D33-Pad1) -> Net-(D33-Pad2)
- SW34 pad 2: Net-(D34-Pad1) -> Net-(D34-Pad2)
- SW35 pad 2: Net-(D35-Pad1) -> Net-(D35-Pad2)
- SW36 pad 2: Net-(D36-Pad1) -> Net-(D36-Pad2)
- SW37 pad 2: Net-(D37-Pad1) -> Net-(D37-Pad2)
- SW38 pad 2: Net-(D38-Pad1) -> Net-(D38-Pad2)
- SW39 pad 2: Net-(D39-Pad1) -> Net-(D39-Pad2)
- SW4 pad 2: Net-(D4-Pad1) -> Net-(D4-Pad2)
- SW40 pad 2: Net-(D40-Pad1) -> Net-(D40-Pad2)
- SW41 pad 2: Net-(D41-Pad1) -> Net-(D41-Pad2)
- SW42 pad 2: Net-(D42-Pad1) -> Net-(D42-Pad2)
- SW43 pad 2: Net-(D43-Pad1) -> Net-(D43-Pad2)
- SW44 pad 2: Net-(D44-Pad1) -> Net-(D44-Pad2)
- SW45 pad 2: Net-(D45-Pad1) -> Net-(D45-Pad2)
- SW46 pad 2: Net-(D46-Pad1) -> Net-(D46-Pad2)
- SW47 pad 2: Net-(D47-Pad1) -> Net-(D47-Pad2)
- SW48 pad 2: Net-(D48-Pad1) -> Net-(D48-Pad2)
- SW49 pad 2: Net-(D49-Pad1) -> Net-(D49-Pad2)
- SW5 pad 2: Net-(D5-Pad1) -> Net-(D5-Pad2)
- SW50 pad 2: Net-(D50-Pad1) -> Net-(D50-Pad2)
- SW51 pad 2: Net-(D51-Pad1) -> Net-(D51-Pad2)
- SW52 pad 2: Net-(D52-Pad1) -> Net-(D52-Pad2)
- SW53 pad 2: Net-(D53-Pad1) -> Net-(D53-Pad2)
- SW54 pad 2: Net-(D54-Pad1) -> Net-(D54-Pad2)
- SW55 pad 2: Net-(D55-Pad1) -> Net-(D55-Pad2)
- SW56 pad 2: Net-(D56-Pad1) -> Net-(D56-Pad2)
- SW57 pad 2: Net-(D57-Pad1) -> Net-(D57-Pad2)
- SW58 pad 2: Net-(D58-Pad1) -> Net-(D58-Pad2)
- SW59 pad 2: Net-(D59-Pad1) -> Net-(D59-Pad2)
- SW6 pad 2: Net-(D6-Pad1) -> Net-(D6-Pad2)
- SW60 pad 2: Net-(D60-Pad1) -> Net-(D60-Pad2)
- SW61 pad 2: Net-(D61-Pad1) -> Net-(D61-Pad2)
- SW62 pad 2: Net-(D62-Pad1) -> Net-(D62-Pad2)
- SW63 pad 2: Net-(D63-Pad1) -> Net-(D63-Pad2)
- SW64 pad 2: Net-(D64-Pad1) -> Net-(D64-Pad2)
- SW66 pad 2: Net-(D66-Pad1) -> Net-(D66-Pad2)
- SW67 pad 2: Net-(D67-Pad1) -> Net-(D67-Pad2)
- SW68 pad 2: Net-(D68-Pad1) -> Net-(D68-Pad2)
- SW69 pad 2: Net-(D69-Pad1) -> Net-(D69-Pad2)
- SW7 pad 2: Net-(D7-Pad1) -> Net-(D7-Pad2)
- SW70 pad 2: Net-(D70-Pad1) -> Net-(D70-Pad2)
- SW71 pad 2: Net-(D71-Pad1) -> Net-(D71-Pad2)
- SW72 pad 2: Net-(D72-Pad1) -> Net-(D72-Pad2)
- SW73 pad 2: Net-(D73-Pad1) -> Net-(D73-Pad2)
- SW74 pad 2: Net-(D74-Pad1) -> Net-(D74-Pad2)
- SW75 pad 2: Net-(D75-Pad1) -> Net-(D75-Pad2)
- SW76 pad 2: Net-(D76-Pad1) -> Net-(D76-Pad2)
- SW77 pad 2: Net-(D77-Pad1) -> Net-(D77-Pad2)
- SW78 pad 2: Net-(D78-Pad1) -> Net-(D78-Pad2)
- SW79 pad 2: Net-(D79-Pad1) -> Net-(D79-Pad2)
- SW8 pad 2: Net-(D8-Pad1) -> Net-(D8-Pad2)
- SW80 pad 2: Net-(D80-Pad1) -> Net-(D80-Pad2)
- SW81 pad 2: Net-(D81-Pad1) -> Net-(D81-Pad2)
- SW82 pad 2: Net-(D82-Pad1) -> Net-(D82-Pad2)
- SW83 pad 2: Net-(D83-Pad1) -> Net-(D83-Pad2)
- SW84 pad 2: Net-(D84-Pad1) -> Net-(D84-Pad2)
- SW85 pad 2: Net-(D85-Pad1) -> Net-(D85-Pad2)
- SW86 pad 2: Net-(D86-Pad1) -> Net-(D86-Pad2)
- SW87 pad 2: Net-(D87-Pad1) -> Net-(D87-Pad2)
- SW88 pad 2: Net-(D88-Pad1) -> Net-(D88-Pad2)
- SW89 pad 2: Net-(D89-Pad1) -> Net-(D89-Pad2)
- SW9 pad 2: Net-(D9-Pad1) -> Net-(D9-Pad2)
- SW90 pad 2: Net-(D90-Pad1) -> Net-(D90-Pad2)
Routing:
- net row04: track 18.4 -> 527.4 mm, vias 0 -> 1
- net row03: track 18.4 -> 518.7 mm
- net row02: track 18.4 -> 516.3 mm, vias 0 -> 2
- net row05: track 18.4 -> 507.6 mm, vias 0 -> 1
- net row01: track 19.4 -> 505.9 mm, vias 0 -> 4
- net col14: track 11.2 -> 489.0 mm, vias 0 -> 5
- net col12: track 12.5 -> 452.3 mm, vias 0 -> 6
- net col13: track 12.3 -> 451.1 mm, vias 0 -> 6
- net col11: track 12.3 -> 437.3 mm, vias 0 -> 6
- net row00: track 18.4 -> 433.6 mm
- net col10: track 12.3 -> 427.5 mm, vias 0 -> 6
- net col09: track 12.3 -> 337.0 mm, vias 0 -> 7
- net col01: track 12.3 -> 335.7 mm, vias 0 -> 3
- net col00: track 17.9 -> 340.3 mm, vias 0 -> 4
- net col08: track 5.62 -> 306.0 mm, vias 0 -> 6
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Other:
- board size 297.2 x 263.7 mm -> 290.9 x 267.8 mm
- board text removed: "74HC595"
- board text removed: "For Left hand"
- board text removed: "For Right hand"

Commit message: 寸法明記 272.00 x 295.00
Parts:
- moved D54 4.47 mm to (255.7, 208.8)
- moved D60 4.47 mm to (252.6, 232.0)
- moved U6 4.47 mm to (252.7, 121.9)
- moved D1 4.47 mm to (141.2, 147.2)
- moved D10 4.47 mm to (151.3, 202.5)
- moved D11 4.47 mm to (148.0, 223.7)
- moved D12 4.47 mm to (155.1, 241.8)
- moved D13 4.47 mm to (179.5, 137.5)
- moved D14 4.47 mm to (172.7, 157.6)
- moved D15 4.47 mm to (172.9, 178.1)
- moved D16 4.47 mm to (170.3, 197.6)
- moved D17 4.47 mm to (167.3, 218.6)
- moved D18 4.47 mm to (174.4, 236.5)
- moved D19 4.47 mm to (198.4, 134.4)
- moved D2 4.47 mm to (134.5, 166.7)
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Routing:
- net row00: track 433.6 -> 437.5 mm
- net col12: track 452.3 -> 449.1 mm
- net row04: track 527.4 -> 526.0 mm
- net col11: track 437.3 -> 435.9 mm
- net col13: track 451.1 -> 449.7 mm
- net col14: track 489.0 -> 487.7 mm
- net col10: track 427.5 -> 426.4 mm
- net row05: track 507.6 -> 506.6 mm
- net Net-(D73-Pad2): track 30.1 -> 29.1 mm
- net VCC: track 190.2 -> 189.3 mm
- net GND: vias 248 -> 268

Commit message: v1.2
Parts:
- SW1, SW10, SW11, SW12, SW13, SW14, SW15, SW16, SW17, SW18, SW19, SW2, SW20, SW21, SW22, SW23, SW24, SW25, SW26, SW27, SW28, SW29, SW3, SW30, SW31, SW32, SW33, SW34, SW35, SW36, SW37, SW38, SW39, SW4, SW40, SW41, SW42, SW43, SW44, SW45, SW46, SW47, SW48, SW5, SW51, SW52, SW53, SW54, SW56, SW57, SW58, SW59, SW6, SW60, SW61, SW62, SW63, SW64, SW65, SW66, SW67, SW68, SW69, SW7, SW70, SW71, SW72, SW73, SW74, SW75, SW76, SW77, SW78, SW79, SW8, SW80, SW81, SW82, SW83, SW84, SW85, SW86, SW87, SW88, SW89, SW9, SW90: footprint kbd:CherryMX_Hotswap -> kbd:CherryMX_Hotswap_edit
- moved D72 49.0 mm to (219.7, 257.0)
- moved D19 49.0 mm to (163.0, 100.5)
- moved D46 48.8 mm to (221.8, 132.2)
- moved D64 48.8 mm to (250.0, 207.4)
- moved D66 48.8 mm to (203.6, 242.2)
- moved D74 48.8 mm to (301.2, 225.9)
- moved D76 48.8 mm to (266.1, 245.9)
- moved D77 48.8 mm to (248.6, 253.8)
- moved D79 48.8 mm to (324.6, 239.8)
- moved D89 48.8 mm to (253.8, 294.6)
- moved HOLE3 48.8 mm to (254.5, 115.2)
- moved SW47 48.8 mm to (245.8, 151.8)
- moved SW48 48.8 mm to (228.6, 163.8)
- moved SW54 48.8 mm to (225.3, 186.1)
- moved SW65 48.8 mm to (232.6, 226.7)
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Routing:
- net col03: track 289.9 -> 276.9 mm, vias 6 -> 7
- net Net-(D72-Pad2): track 37.5 -> 26.0 mm, vias 0 -> 1
- net col13: track 449.7 -> 460.5 mm
- net Net-(D1-Pad2): track 37.6 -> 29.0 mm
- net row05: track 506.6 -> 515.0 mm, vias 1 -> 0
- net row03: track 518.7 -> 527.0 mm, vias 0 -> 1
- net col11: track 435.9 -> 444.1 mm
- net Net-(D18-Pad2): track 31.9 -> 24.1 mm, vias 0 -> 1
- net col09: track 337.0 -> 344.7 mm
- net Net-(D66-Pad2): track 35.1 -> 27.4 mm, vias 0 -> 1
- net hardware_reset: track 38.4 -> 46.1 mm
- net col12: track 449.1 -> 456.6 mm
- net software_reset: track 68.7 -> 75.9 mm
- net col05: track 263.3 -> 270.3 mm
- net col00: track 340.3 -> 345.6 mm
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Other:
- rule trace_min: 0.2 -> 0
