File: fan/fan.kicad_pcb (KiCad board)
At the start: 2 copper layers, 290.9 x 267.8 mm, 196 parts, among them J2 Pi, SW1 SW_PUSH, SW10 SW_PUSH, SW11 SW_PUSH, SW12 SW_PUSH, SW13 SW_PUSH, SW14 SW_PUSH, SW15 SW_PUSH, SW16 SW_PUSH, SW17 SW_PUSH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

Commit message: v1.21
Other:
- rule trace_min: 0 -> 0.2

Commit message: 発注した
Parts:
- J2: footprint Connector_PinSocket_2.54mm:PinSocket_2x20_P2.54mm_Vertical -> kbd:PinSocket_2x20_P2.54mm_Vertical_edit
- SW93: footprint Button_Switch_THT:SW_Slide_1P2T_CK_OS102011MS2Q -> kbd:SW_Slide_edit
