File: fan/fan.kicad_pcb (KiCad board)
At the start: 2 copper layers, 290.9 x 267.8 mm, 196 parts, among them J2 Pi, SW1 SW_PUSH, SW10 SW_PUSH, SW11 SW_PUSH, SW12 SW_PUSH, SW13 SW_PUSH, SW14 SW_PUSH, SW15 SW_PUSH, SW16 SW_PUSH, SW17 SW_PUSH, SW18 SW_PUSH, SW19 SW_PUSH, SW2 SW_PUSH, SW20 SW_PUSH, SW21 SW_PUSH, SW22 SW_PUSH, SW23 SW_PUSH, SW24 SW_PUSH, SW25 SW_PUSH, SW26 SW_PUSH, SW27 SW_PUSH, SW28 SW_PUSH, SW29 SW_PUSH, SW3 SW_PUSH, SW30 SW_PUSH, SW31 SW_PUSH, SW32 SW_PUSH, SW33 SW_PUSH, SW34 SW_PUSH, SW35 SW_PUSH, SW36 SW_PUSH, SW37 SW_PUSH, SW38 SW_PUSH, SW39 SW_PUSH, SW4 SW_PUSH, SW40 SW_PUSH, SW41 SW_PUSH, SW42 SW_PUSH, SW43 SW_PUSH, SW44 SW_PUSH, SW45 SW_PUSH, SW46 SW_PUSH, SW47 SW_PUSH, SW48 SW_PUSH, SW49 SW_PUSH, SW5 SW_PUSH, SW50 SW_PUSH, SW51 SW_PUSH, SW52 SW_PUSH, SW53 SW_PUSH, SW54 SW_PUSH, SW55 SW_PUSH, SW56 SW_PUSH, SW57 SW_PUSH, SW58 SW_PUSH, SW59 SW_PUSH, SW6 SW_PUSH, SW60 SW_PUSH, SW61 SW_PUSH, SW62 SW_PUSH, SW63 SW_PUSH, SW64 SW_PUSH, SW65 SW_PUSH, SW66 SW_PUSH, SW67 SW_PUSH, SW68 SW_PUSH, SW69 SW_PUSH, SW7 SW_PUSH, SW70 SW_PUSH, SW71 SW_PUSH, SW72 SW_PUSH, SW73 SW_PUSH, SW74 SW_PUSH, SW75 SW_PUSH, SW76 SW_PUSH, SW77 SW_PUSH, SW78 SW_PUSH, SW79 SW_PUSH, SW8 SW_PUSH, SW80 SW_PUSH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

Commit message: アクリルレーザーカット用ファイルを追加
Parts:
- moved D85 86.9 mm to (266.5, 198.8)
- moved D50 86.9 mm to (225.5, 89.4)
- moved HOLE5 86.9 mm to (283.1, 210.4)
- moved SW52 86.9 mm to (199.2, 106.0)
- moved SW58 86.9 mm to (195.3, 132.7)
- moved SW77 86.9 mm to (183.7, 204.4)
- moved SW78 86.9 mm to (160.4, 210.0)
- moved D34 86.9 mm to (118.3, 97.8)
- moved SW57 86.9 mm to (211.3, 121.9)
- moved SW80 86.9 mm to (241.3, 196.1)
- moved D10 86.9 mm to (53.8, 108.1)
- moved D12 86.9 mm to (57.6, 147.4)
- moved D13 86.9 mm to (82.0, 43.1)
- moved D14 86.9 mm to (75.2, 63.2)
- moved D15 86.9 mm to (75.5, 83.7)
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Connections:
- D1 pad 1: row00 -> (no net)
- D1 pad 2: Net-(D1-Pad2) -> (no net)
- D10 pad 1: row03 -> (no net)
- D10 pad 2: Net-(D10-Pad2) -> (no net)
- D11 pad 1: row04 -> (no net)
- D11 pad 2: Net-(D11-Pad2) -> (no net)
- D12 pad 1: row05 -> (no net)
- D12 pad 2: Net-(D12-Pad2) -> (no net)
- D13 pad 1: row00 -> (no net)
- D13 pad 2: Net-(D13-Pad2) -> (no net)
- D14 pad 1: row01 -> (no net)
- D14 pad 2: Net-(D14-Pad2) -> (no net)
- D15 pad 1: row02 -> (no net)
- D15 pad 2: Net-(D15-Pad2) -> (no net)
- D16 pad 1: row03 -> (no net)
- D16 pad 2: Net-(D16-Pad2) -> (no net)
- D17 pad 1: row04 -> (no net)
- D17 pad 2: Net-(D17-Pad2) -> (no net)
- D18 pad 1: row05 -> (no net)
- D18 pad 2: Net-(D18-Pad2) -> (no net)
- D19 pad 1: row00 -> (no net)
- D19 pad 2: Net-(D19-Pad2) -> (no net)
- D2 pad 1: row01 -> (no net)
- D2 pad 2: Net-(D2-Pad2) -> (no net)
- D20 pad 1: row01 -> (no net)
- D20 pad 2: Net-(D20-Pad2) -> (no net)
- D21 pad 1: row02 -> (no net)
- D21 pad 2: Net-(D21-Pad2) -> (no net)
- D22 pad 1: row03 -> (no net)
- D22 pad 2: Net-(D22-Pad2) -> (no net)
- D23 pad 1: row04 -> (no net)
- D23 pad 2: Net-(D23-Pad2) -> (no net)
- D24 pad 1: row05 -> (no net)
- D24 pad 2: Net-(D24-Pad2) -> (no net)
- D25 pad 1: row00 -> (no net)
- D25 pad 2: Net-(D25-Pad2) -> (no net)
- D26 pad 1: row01 -> (no net)
- D26 pad 2: Net-(D26-Pad2) -> (no net)
- D27 pad 1: row02 -> (no net)
- D27 pad 2: Net-(D27-Pad2) -> (no net)
- D28 pad 1: row03 -> (no net)
- D28 pad 2: Net-(D28-Pad2) -> (no net)
- D29 pad 1: row04 -> (no net)
- D29 pad 2: Net-(D29-Pad2) -> (no net)
- D3 pad 1: row02 -> (no net)
- D3 pad 2: Net-(D3-Pad2) -> (no net)
- D30 pad 1: row05 -> (no net)
- D30 pad 2: Net-(D30-Pad2) -> (no net)
- D31 pad 1: row00 -> (no net)
- D31 pad 2: Net-(D31-Pad2) -> (no net)
- D32 pad 1: row01 -> (no net)
- D32 pad 2: Net-(D32-Pad2) -> (no net)
- D33 pad 1: row02 -> (no net)
- D33 pad 2: Net-(D33-Pad2) -> (no net)
- D34 pad 1: row03 -> (no net)
- D34 pad 2: Net-(D34-Pad2) -> (no net)
- D35 pad 1: row04 -> (no net)
- D35 pad 2: Net-(D35-Pad2) -> (no net)
- D36 pad 1: row05 -> (no net)
- D36 pad 2: Net-(D36-Pad2) -> (no net)
- D37 pad 1: row00 -> (no net)
- D37 pad 2: Net-(D37-Pad2) -> (no net)
- D38 pad 1: row01 -> (no net)
- D38 pad 2: Net-(D38-Pad2) -> (no net)
- D39 pad 1: row02 -> (no net)
- D39 pad 2: Net-(D39-Pad2) -> (no net)
- D4 pad 1: row03 -> (no net)
- D4 pad 2: Net-(D4-Pad2) -> (no net)
- D40 pad 1: row03 -> (no net)
- D40 pad 2: Net-(D40-Pad2) -> (no net)
- D41 pad 1: row04 -> (no net)
- D41 pad 2: Net-(D41-Pad2) -> (no net)
- D42 pad 1: row05 -> (no net)
- D42 pad 2: Net-(D42-Pad2) -> (no net)
- D43 pad 1: row00 -> (no net)
- D43 pad 2: Net-(D43-Pad2) -> (no net)
- D44 pad 1: row01 -> (no net)
- D44 pad 2: Net-(D44-Pad2) -> (no net)
- D45 pad 1: row02 -> (no net)
- D45 pad 2: Net-(D45-Pad2) -> (no net)
- D46 pad 1: row03 -> (no net)
- D46 pad 2: Net-(D46-Pad2) -> (no net)
- D47 pad 1: row04 -> (no net)
- D47 pad 2: Net-(D47-Pad2) -> (no net)
- D48 pad 1: row05 -> (no net)
- D48 pad 2: Net-(D48-Pad2) -> (no net)
- D49 pad 1: row00 -> (no net)
- D49 pad 2: Net-(D49-Pad2) -> (no net)
- D5 pad 1: row04 -> (no net)
- D5 pad 2: Net-(D5-Pad2) -> (no net)
- D50 pad 1: row01 -> (no net)
- D50 pad 2: Net-(D50-Pad2) -> (no net)
- D51 pad 1: row02 -> (no net)
- D51 pad 2: Net-(D51-Pad2) -> (no net)
- D52 pad 1: row03 -> (no net)
- D52 pad 2: Net-(D52-Pad2) -> (no net)
- D53 pad 1: row04 -> (no net)
- D53 pad 2: Net-(D53-Pad2) -> (no net)
- D54 pad 1: row05 -> (no net)
- D54 pad 2: Net-(D54-Pad2) -> (no net)
- D55 pad 1: row00 -> (no net)
- D55 pad 2: Net-(D55-Pad2) -> (no net)
- D56 pad 1: row01 -> (no net)
- D56 pad 2: Net-(D56-Pad2) -> (no net)
- D57 pad 1: row02 -> (no net)
- D57 pad 2: Net-(D57-Pad2) -> (no net)
- D58 pad 1: row03 -> (no net)
- D58 pad 2: Net-(D58-Pad2) -> (no net)
- D59 pad 1: row04 -> (no net)
- D59 pad 2: Net-(D59-Pad2) -> (no net)
- D6 pad 1: row05 -> (no net)
- D6 pad 2: Net-(D6-Pad2) -> (no net)
- D60 pad 1: row05 -> (no net)
- D60 pad 2: Net-(D60-Pad2) -> (no net)
- D61 pad 1: row00 -> (no net)
- D61 pad 2: Net-(D61-Pad2) -> (no net)
- D62 pad 1: row01 -> (no net)
- D62 pad 2: Net-(D62-Pad2) -> (no net)
- D63 pad 1: row02 -> (no net)
- D63 pad 2: Net-(D63-Pad2) -> (no net)
- D64 pad 1: row03 -> (no net)
- D64 pad 2: Net-(D64-Pad2) -> (no net)
- D65 pad 1: row04 -> (no net)
- D65 pad 2: Net-(D65-Pad2) -> (no net)
- D66 pad 1: row05 -> (no net)
- D66 pad 2: Net-(D66-Pad2) -> (no net)
- D67 pad 1: row00 -> (no net)
- D67 pad 2: Net-(D67-Pad2) -> (no net)
- D68 pad 1: row01 -> (no net)
- D68 pad 2: Net-(D68-Pad2) -> (no net)
- D69 pad 1: row02 -> (no net)
- D69 pad 2: Net-(D69-Pad2) -> (no net)
- D7 pad 1: row00 -> (no net)
- D7 pad 2: Net-(D7-Pad2) -> (no net)
- D70 pad 1: row03 -> (no net)
- D70 pad 2: Net-(D70-Pad2) -> (no net)
- D71 pad 1: row04 -> (no net)
- D71 pad 2: Net-(D71-Pad2) -> (no net)
- D72 pad 1: row05 -> (no net)
- D72 pad 2: Net-(D72-Pad2) -> (no net)
- D73 pad 1: row00 -> (no net)
- D73 pad 2: Net-(D73-Pad2) -> (no net)
- D74 pad 1: row01 -> (no net)
- D74 pad 2: Net-(D74-Pad2) -> (no net)
- D75 pad 1: row02 -> (no net)
- D75 pad 2: Net-(D75-Pad2) -> (no net)
- D76 pad 1: row03 -> (no net)
- D76 pad 2: Net-(D76-Pad2) -> (no net)
- D77 pad 1: row04 -> (no net)
- D77 pad 2: Net-(D77-Pad2) -> (no net)
- D78 pad 1: row05 -> (no net)
- D78 pad 2: Net-(D78-Pad2) -> (no net)
- D79 pad 1: row00 -> (no net)
- D79 pad 2: Net-(D79-Pad2) -> (no net)
- D8 pad 1: row01 -> (no net)
- D8 pad 2: Net-(D8-Pad2) -> (no net)
- D80 pad 1: row01 -> (no net)
- D80 pad 2: Net-(D80-Pad2) -> (no net)
- D81 pad 1: row02 -> (no net)
- D81 pad 2: Net-(D81-Pad2) -> (no net)
- D82 pad 1: row03 -> (no net)
- D82 pad 2: Net-(D82-Pad2) -> (no net)
- D83 pad 1: row04 -> (no net)
- D83 pad 2: Net-(D83-Pad2) -> (no net)
- D84 pad 1: row05 -> (no net)
- D84 pad 2: Net-(D84-Pad2) -> (no net)
- D85 pad 1: row00 -> (no net)
- D85 pad 2: Net-(D85-Pad2) -> (no net)
- D86 pad 1: row01 -> (no net)
- D86 pad 2: Net-(D86-Pad2) -> (no net)
- D87 pad 1: row02 -> (no net)
- D87 pad 2: Net-(D87-Pad2) -> (no net)
- D88 pad 1: row03 -> (no net)
- D88 pad 2: Net-(D88-Pad2) -> (no net)
- D89 pad 1: row04 -> (no net)
- D89 pad 2: Net-(D89-Pad2) -> (no net)
- D9 pad 1: row02 -> (no net)
- D9 pad 2: Net-(D9-Pad2) -> (no net)
- D90 pad 1: row05 -> (no net)
- D90 pad 2: Net-(D90-Pad2) -> (no net)
- J2 pad 36: GND -> (no net)
- J2 pad 38: Net-(J2-Pad38) -> (no net)
- J2 pad 40: Net-(J2-Pad38) -> (no net)
- SW1 pad 1: col00 -> (no net)
- SW1 pad 2: Net-(D1-Pad2) -> (no net)
- SW10 pad 1: col01 -> (no net)
- SW10 pad 2: Net-(D10-Pad2) -> (no net)
- SW11 pad 1: col01 -> (no net)
- SW11 pad 2: Net-(D11-Pad2) -> (no net)
- SW12 pad 1: col01 -> (no net)
- SW12 pad 2: Net-(D12-Pad2) -> (no net)
- SW13 pad 1: col02 -> (no net)
- SW13 pad 2: Net-(D13-Pad2) -> (no net)
- SW14 pad 1: col02 -> (no net)
- SW14 pad 2: Net-(D14-Pad2) -> (no net)
- SW15 pad 1: col02 -> (no net)
- SW15 pad 2: Net-(D15-Pad2) -> (no net)
- SW16 pad 1: col02 -> (no net)
- SW16 pad 2: Net-(D16-Pad2) -> (no net)
- SW17 pad 1: col02 -> (no net)
- SW17 pad 2: Net-(D17-Pad2) -> (no net)
- SW18 pad 1: col02 -> (no net)
- SW18 pad 2: Net-(D18-Pad2) -> (no net)
- SW19 pad 1: col03 -> (no net)
- SW19 pad 2: Net-(D19-Pad2) -> (no net)
- SW2 pad 1: col00 -> (no net)
- SW2 pad 2: Net-(D2-Pad2) -> (no net)
- SW20 pad 1: col03 -> (no net)
- SW20 pad 2: Net-(D20-Pad2) -> (no net)
- SW21 pad 1: col03 -> (no net)
- SW21 pad 2: Net-(D21-Pad2) -> (no net)
- SW22 pad 1: col03 -> (no net)
- SW22 pad 2: Net-(D22-Pad2) -> (no net)
- SW23 pad 1: col03 -> (no net)
- SW23 pad 2: Net-(D23-Pad2) -> (no net)
- SW24 pad 1: col03 -> (no net)
- SW24 pad 2: Net-(D24-Pad2) -> (no net)
- SW25 pad 1: col04 -> (no net)
- SW25 pad 2: Net-(D25-Pad2) -> (no net)
- SW26 pad 1: col04 -> (no net)
- SW26 pad 2: Net-(D26-Pad2) -> (no net)
- SW27 pad 1: col04 -> (no net)
- SW27 pad 2: Net-(D27-Pad2) -> (no net)
- SW28 pad 1: col04 -> (no net)
- SW28 pad 2: Net-(D28-Pad2) -> (no net)
- SW29 pad 1: col04 -> (no net)
- SW29 pad 2: Net-(D29-Pad2) -> (no net)
- SW3 pad 1: col00 -> (no net)
- SW3 pad 2: Net-(D3-Pad2) -> (no net)
- SW30 pad 1: col04 -> (no net)
- SW30 pad 2: Net-(D30-Pad2) -> (no net)
- SW31 pad 1: col05 -> (no net)
- SW31 pad 2: Net-(D31-Pad2) -> (no net)
- SW32 pad 1: col05 -> (no net)
- SW32 pad 2: Net-(D32-Pad2) -> (no net)
- SW33 pad 1: col05 -> (no net)
- SW33 pad 2: Net-(D33-Pad2) -> (no net)
- SW34 pad 1: col05 -> (no net)
- SW34 pad 2: Net-(D34-Pad2) -> (no net)
- SW35 pad 1: col05 -> (no net)
- SW35 pad 2: Net-(D35-Pad2) -> (no net)
- SW36 pad 1: col05 -> (no net)
- SW36 pad 2: Net-(D36-Pad2) -> (no net)
- SW37 pad 1: col06 -> (no net)
- SW37 pad 2: Net-(D37-Pad2) -> (no net)
- SW38 pad 1: col06 -> (no net)
- SW38 pad 2: Net-(D38-Pad2) -> (no net)
- SW39 pad 1: col06 -> (no net)
- SW39 pad 2: Net-(D39-Pad2) -> (no net)
- SW4 pad 1: col00 -> (no net)
- SW4 pad 2: Net-(D4-Pad2) -> (no net)
- SW40 pad 1: col06 -> (no net)
- SW40 pad 2: Net-(D40-Pad2) -> (no net)
- SW41 pad 1: col06 -> (no net)
- SW41 pad 2: Net-(D41-Pad2) -> (no net)
- SW42 pad 1: col06 -> (no net)
- SW42 pad 2: Net-(D42-Pad2) -> (no net)
- SW43 pad 1: col07 -> (no net)
- SW43 pad 2: Net-(D43-Pad2) -> (no net)
- SW44 pad 1: col07 -> (no net)
- SW44 pad 2: Net-(D44-Pad2) -> (no net)
- SW45 pad 1: col07 -> (no net)
- SW45 pad 2: Net-(D45-Pad2) -> (no net)
- SW46 pad 1: col07 -> (no net)
- SW46 pad 2: Net-(D46-Pad2) -> (no net)
- SW47 pad 1: col07 -> (no net)
- SW47 pad 2: Net-(D47-Pad2) -> (no net)
- SW48 pad 1: col07 -> (no net)
- SW48 pad 2: Net-(D48-Pad2) -> (no net)
- SW49 pad 1: col08 -> (no net)
- SW49 pad 2: Net-(D49-Pad2) -> (no net)
- SW5 pad 1: col00 -> (no net)
- SW5 pad 2: Net-(D5-Pad2) -> (no net)
- SW50 pad 1: col08 -> (no net)
- SW50 pad 2: Net-(D50-Pad2) -> (no net)
- SW51 pad 1: col08 -> (no net)
- SW51 pad 2: Net-(D51-Pad2) -> (no net)
- SW52 pad 1: col08 -> (no net)
- SW52 pad 2: Net-(D52-Pad2) -> (no net)
- SW53 pad 1: col08 -> (no net)
- SW53 pad 2: Net-(D53-Pad2) -> (no net)
- SW54 pad 1: col08 -> (no net)
- SW54 pad 2: Net-(D54-Pad2) -> (no net)
- SW55 pad 1: col09 -> (no net)
- SW55 pad 2: Net-(D55-Pad2) -> (no net)
- SW56 pad 1: col09 -> (no net)
- SW56 pad 2: Net-(D56-Pad2) -> (no net)
- SW57 pad 1: col09 -> (no net)
- SW57 pad 2: Net-(D57-Pad2) -> (no net)
- SW58 pad 1: col09 -> (no net)
- SW58 pad 2: Net-(D58-Pad2) -> (no net)
- SW59 pad 1: col09 -> (no net)
- SW59 pad 2: Net-(D59-Pad2) -> (no net)
- SW6 pad 1: col00 -> (no net)
- SW6 pad 2: Net-(D6-Pad2) -> (no net)
- SW60 pad 1: col09 -> (no net)
- SW60 pad 2: Net-(D60-Pad2) -> (no net)
- SW61 pad 1: col10 -> (no net)
- SW61 pad 2: Net-(D61-Pad2) -> (no net)
- SW62 pad 1: col10 -> (no net)
- SW62 pad 2: Net-(D62-Pad2) -> (no net)
- SW63 pad 1: col10 -> (no net)
- SW63 pad 2: Net-(D63-Pad2) -> (no net)
- SW64 pad 1: col10 -> (no net)
- SW64 pad 2: Net-(D64-Pad2) -> (no net)
- SW65 pad 1: col10 -> (no net)
- SW65 pad 2: Net-(D65-Pad2) -> (no net)
- SW66 pad 1: col10 -> (no net)
- SW66 pad 2: Net-(D66-Pad2) -> (no net)
- SW67 pad 1: col11 -> (no net)
- SW67 pad 2: Net-(D67-Pad2) -> (no net)
- SW68 pad 1: col11 -> (no net)
- SW68 pad 2: Net-(D68-Pad2) -> (no net)
- SW69 pad 1: col11 -> (no net)
- SW69 pad 2: Net-(D69-Pad2) -> (no net)
- SW7 pad 1: col01 -> (no net)
- SW7 pad 2: Net-(D7-Pad2) -> (no net)
- SW70 pad 1: col11 -> (no net)
- SW70 pad 2: Net-(D70-Pad2) -> (no net)
- SW71 pad 1: col11 -> (no net)
- SW71 pad 2: Net-(D71-Pad2) -> (no net)
- SW72 pad 1: col11 -> (no net)
- SW72 pad 2: Net-(D72-Pad2) -> (no net)
- SW73 pad 1: col12 -> (no net)
- SW73 pad 2: Net-(D73-Pad2) -> (no net)
- SW74 pad 1: col12 -> (no net)
- SW74 pad 2: Net-(D74-Pad2) -> (no net)
- SW75 pad 1: col12 -> (no net)
- SW75 pad 2: Net-(D75-Pad2) -> (no net)
- SW76 pad 1: col12 -> (no net)
- SW76 pad 2: Net-(D76-Pad2) -> (no net)
- SW77 pad 1: col12 -> (no net)
- SW77 pad 2: Net-(D77-Pad2) -> (no net)
- SW78 pad 1: col12 -> (no net)
- SW78 pad 2: Net-(D78-Pad2) -> (no net)
- SW79 pad 1: col13 -> (no net)
- SW79 pad 2: Net-(D79-Pad2) -> (no net)
- SW8 pad 1: col01 -> (no net)
- SW8 pad 2: Net-(D8-Pad2) -> (no net)
- SW80 pad 1: col13 -> (no net)
- SW80 pad 2: Net-(D80-Pad2) -> (no net)
- SW81 pad 1: col13 -> (no net)
- SW81 pad 2: Net-(D81-Pad2) -> (no net)
- SW82 pad 1: col13 -> (no net)
- SW82 pad 2: Net-(D82-Pad2) -> (no net)
- SW83 pad 1: col13 -> (no net)
- SW83 pad 2: Net-(D83-Pad2) -> (no net)
- SW84 pad 1: col13 -> (no net)
- SW84 pad 2: Net-(D84-Pad2) -> (no net)
- SW85 pad 1: col14 -> (no net)
- SW85 pad 2: Net-(D85-Pad2) -> (no net)
- SW86 pad 1: col14 -> (no net)
- SW86 pad 2: Net-(D86-Pad2) -> (no net)
- SW87 pad 1: col14 -> (no net)
- SW87 pad 2: Net-(D87-Pad2) -> (no net)
- SW88 pad 1: col14 -> (no net)
- SW88 pad 2: Net-(D88-Pad2) -> (no net)
- SW89 pad 1: col14 -> (no net)
- SW89 pad 2: Net-(D89-Pad2) -> (no net)
- SW9 pad 1: col01 -> (no net)
- SW9 pad 2: Net-(D9-Pad2) -> (no net)
- SW90 pad 1: col14 -> (no net)
- SW90 pad 2: Net-(D90-Pad2) -> (no net)
- SW91 pad 1: software_reset -> (no net)
- SW91 pad 2: GND -> (no net)
- SW92 pad 1: hardware_reset -> (no net)
- SW92 pad 2: GND -> (no net)
- SW93 pad 2: Net-(J2-Pad38) -> (no net)
- SW93 pad 3: VCC -> (no net)
- U1 pad 10: SCL -> (no net)
- U1 pad 11: RCK -> (no net)
- U1 pad 12: OE -> (no net)
- U1 pad 13: row05 -> (no net)
- U1 pad 14: row04 -> (no net)
- U1 pad 15: row03 -> (no net)
- U1 pad 16: row02 -> (no net)
- U1 pad 17: row01 -> (no net)
- U1 pad 18: row00 -> (no net)
- U1 pad 21: VCC -> (no net)
- U1 pad 22: hardware_reset -> (no net)
- U1 pad 23: GND -> (no net)
- U1 pad 3: GND -> (no net)
- U1 pad 4: GND -> (no net)
- U1 pad 7: software_reset -> (no net)
- U1 pad 8: SER -> (no net)
- U1 pad 9: SCK -> (no net)
- U2 pad 10: SCL -> (no net)
- U2 pad 11: RCK -> (no net)
- U2 pad 12: OE -> (no net)
- U2 pad 13: row05 -> (no net)
- U2 pad 14: row04 -> (no net)
- U2 pad 15: row03 -> (no net)
- U2 pad 16: row02 -> (no net)
- U2 pad 17: row01 -> (no net)
- U2 pad 18: row00 -> (no net)
- U2 pad 21: VCC -> (no net)
- U2 pad 22: hardware_reset -> (no net)
- U2 pad 23: GND -> (no net)
- U2 pad 3: GND -> (no net)
- U2 pad 4: GND -> (no net)
- U2 pad 7: software_reset -> (no net)
- U2 pad 8: SER -> (no net)
- U2 pad 9: SCK -> (no net)
- U3 pad 1: col01 -> (no net)
- U3 pad 10: SCL -> (no net)
- U3 pad 11: SCK -> (no net)
- U3 pad 12: RCK -> (no net)
- U3 pad 13: OE -> (no net)
- U3 pad 14: SER -> (no net)
- U3 pad 15: col00 -> (no net)
- U3 pad 16: VCC -> (no net)
- U3 pad 2: col02 -> (no net)
- U3 pad 3: col03 -> (no net)
- U3 pad 4: col04 -> (no net)
- U3 pad 5: col05 -> (no net)
- U3 pad 6: col06 -> (no net)
- U3 pad 7: col07 -> (no net)
- U3 pad 8: GND -> (no net)
- U3 pad 9: QHSER -> (no net)
- U4 pad 1: col09 -> (no net)
- U4 pad 10: SCL -> (no net)
- U4 pad 11: SCK -> (no net)
- U4 pad 12: RCK -> (no net)
- U4 pad 13: OE -> (no net)
- U4 pad 14: QHSER -> (no net)
- U4 pad 15: col08 -> (no net)
- U4 pad 16: VCC -> (no net)
- U4 pad 2: col10 -> (no net)
- U4 pad 3: col11 -> (no net)
- U4 pad 4: col12 -> (no net)
- U4 pad 5: col13 -> (no net)
- U4 pad 6: col14 -> (no net)
- U4 pad 8: GND -> (no net)
- U5 pad 1: col01 -> (no net)
- U5 pad 10: SCL -> (no net)
- U5 pad 11: SCK -> (no net)
- U5 pad 12: RCK -> (no net)
- U5 pad 13: OE -> (no net)
- U5 pad 14: SER -> (no net)
- U5 pad 15: col00 -> (no net)
- U5 pad 16: VCC -> (no net)
- U5 pad 2: col02 -> (no net)
- U5 pad 3: col03 -> (no net)
- U5 pad 4: col04 -> (no net)
- U5 pad 5: col05 -> (no net)
- U5 pad 6: col06 -> (no net)
- U5 pad 7: col07 -> (no net)
- U5 pad 8: GND -> (no net)
- U5 pad 9: QHSER' -> (no net)
- U6 pad 1: col09 -> (no net)
- U6 pad 10: SCL -> (no net)
- U6 pad 11: SCK -> (no net)
- U6 pad 12: RCK -> (no net)
- U6 pad 13: OE -> (no net)
- U6 pad 14: QHSER' -> (no net)
- U6 pad 15: col08 -> (no net)
- U6 pad 16: VCC -> (no net)
- U6 pad 2: col10 -> (no net)
- U6 pad 3: col11 -> (no net)
- U6 pad 4: col12 -> (no net)
- U6 pad 5: col13 -> (no net)
- U6 pad 6: col14 -> (no net)
- U6 pad 8: GND -> (no net)
Routing:
- net (no net): track 0.00 -> 11725.6 mm, vias 0 -> 448
- net row03: track 527.0 -> 0.00 mm, vias 1 -> 0
- net row04: track 521.0 -> 0.00 mm, vias 1 -> 0
- net row02: track 517.0 -> 0.00 mm, vias 2 -> 0
- net row05: track 515.0 -> 0.00 mm
- net row01: track 509.3 -> 0.00 mm, vias 4 -> 0
- net col14: track 489.3 -> 0.00 mm, vias 5 -> 0
- net col13: track 460.4 -> 0.00 mm, vias 6 -> 0
- net col12: track 456.5 -> 0.00 mm, vias 6 -> 0
- net col11: track 444.0 -> 0.00 mm, vias 6 -> 0
- net row00: track 438.8 -> 0.00 mm
- net col10: track 423.6 -> 0.00 mm, vias 6 -> 0
- net col00: track 345.6 -> 0.00 mm, vias 4 -> 0
- net col09: track 344.7 -> 0.00 mm, vias 7 -> 0
- net col01: track 338.8 -> 0.00 mm, vias 3 -> 0
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- added copper zone on B.Cu, net (none)
- added copper zone on F.Cu, net (none)
- removed copper zone on B.Cu, net GND
- removed copper zone on F.Cu, net GND

Commit message: アクリルカットサービスに見積もり出した
Parts:
- J2: footprint kbd:PinSocket_2x20_P2.54mm_Vertical_edit -> kbd:PinSocket_2x20_P2.54mm_Vertical_edit_wakunasi
- SW1, SW10, SW11, SW12, SW13, SW14, SW15, SW16, SW17, SW18, SW19, SW2, SW20, SW21, SW22, SW23, SW24, SW25, SW26, SW27, SW28, SW29, SW3, SW30, SW31, SW32, SW33, SW34, SW35, SW36, SW37, SW38, SW39, SW4, SW40, SW41, SW42, SW43, SW44, SW45, SW46, SW47, SW48, SW5, SW51, SW52, SW53, SW54, SW56, SW57, SW58, SW59, SW6, SW60, SW61, SW62, SW63, SW64, SW65, SW66, SW67, SW68, SW69, SW7, SW70, SW71, SW72, SW73, SW74, SW75, SW76, SW77, SW78, SW79, SW8, SW80, SW81, SW82, SW83, SW84, SW85, SW86, SW87, SW88, SW89, SW9, SW90: footprint kbd:CherryMX_Hotswap_edit -> kbd:CherryMX_Hotswap_edit_wakunasi
- SW49, SW50, SW55, SW91, SW92: footprint kbd:ResetSW -> kbd:ResetSW_wakunasi
- SW93: footprint kbd:SW_Slide_edit -> kbd:SW_Slide_edit_wakunasi
- moved SW73 14.1 mm to (265.1, 181.0)
- moved D23 14.1 mm to (99.4, 129.4)
- moved D30 14.1 mm to (130.5, 149.6)
- moved SW35 14.1 mm to (132.7, 135.1)
- moved D12 14.1 mm to (67.6, 157.4)
- moved D44 14.1 mm to (193.8, 71.1)
- moved HOLE1 14.1 mm to (35.3, 45.5)
- moved SW17 14.1 mm to (71.4, 141.3)
- moved SW2 14.1 mm to (38.9, 89.8)
- moved SW45 14.1 mm to (182.3, 70.5)
- moved SW5 14.1 mm to (34.3, 153.5)
- moved D1 14.1 mm to (53.8, 62.8)
- moved D10 14.1 mm to (63.8, 118.1)
- moved D11 14.1 mm to (60.6, 139.3)
- moved D13 14.1 mm to (92.0, 53.1)
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