File: fan/fan_case/fan_case.kicad_pcb (KiCad board)
At the start: 2 copper layers, 277.7 x 277.4 mm, 196 parts, among them J2 Pi, SW1 SW_PUSH, SW10 SW_PUSH, SW11 SW_PUSH, SW12 SW_PUSH, SW13 SW_PUSH, SW14 SW_PUSH, SW15 SW_PUSH, SW16 SW_PUSH, SW17 SW_PUSH, SW18 SW_PUSH, SW19 SW_PUSH, SW2 SW_PUSH, SW20 SW_PUSH, SW21 SW_PUSH, SW22 SW_PUSH, SW23 SW_PUSH, SW24 SW_PUSH, SW25 SW_PUSH, SW26 SW_PUSH, SW27 SW_PUSH, SW28 SW_PUSH, SW29 SW_PUSH, SW3 SW_PUSH, SW30 SW_PUSH, SW31 SW_PUSH, SW32 SW_PUSH, SW33 SW_PUSH, SW34 SW_PUSH, SW35 SW_PUSH, SW36 SW_PUSH, SW37 SW_PUSH, SW38 SW_PUSH, SW39 SW_PUSH, SW4 SW_PUSH, SW40 SW_PUSH, SW41 SW_PUSH, SW42 SW_PUSH, SW43 SW_PUSH, SW44 SW_PUSH, SW45 SW_PUSH, SW46 SW_PUSH, SW47 SW_PUSH, SW48 SW_PUSH, SW49 SW_PUSH, SW5 SW_PUSH, SW50 SW_PUSH, SW51 SW_PUSH, SW52 SW_PUSH, SW53 SW_PUSH, SW54 SW_PUSH, SW55 SW_PUSH, SW56 SW_PUSH, SW57 SW_PUSH, SW58 SW_PUSH, SW59 SW_PUSH, SW6 SW_PUSH, SW60 SW_PUSH, SW61 SW_PUSH, SW62 SW_PUSH, SW63 SW_PUSH, SW64 SW_PUSH, SW65 SW_PUSH, SW66 SW_PUSH, SW67 SW_PUSH, SW68 SW_PUSH, SW69 SW_PUSH, SW7 SW_PUSH, SW70 SW_PUSH, SW71 SW_PUSH, SW72 SW_PUSH, SW73 SW_PUSH, SW74 SW_PUSH, SW75 SW_PUSH, SW76 SW_PUSH, SW77 SW_PUSH, SW78 SW_PUSH, SW79 SW_PUSH, SW8 SW_PUSH, SW80 SW_PUSH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

Commit message: アクリルパーツをフットプリントにしている最中 あと一つ大きなフタのみ
Parts:
- added REF**: L_case_parts, kbd:L_case_parts, F.Cu at (294.0, 50.0)
- added REF**: L_case_parts, kbd:L_case_parts, F.Cu at (33.0, 290.0)
- added REF**: washer, kbd:washer, F.Cu at (90.0, 264.2)
- added REF**: washer, kbd:washer, F.Cu at (90.0, 282.2)
- added REF**: washer, kbd:washer, F.Cu at (82.0, 282.3)
- added REF**: washer, kbd:washer, F.Cu at (82.0, 273.3)
- added REF**: washer, kbd:washer, F.Cu at (90.0, 273.2)
- added REF**: washer, kbd:washer, F.Cu at (82.0, 264.3)
- added REF**: washer, kbd:washer, F.Cu at (90.1, 255.4)
- added REF**: washer, kbd:washer, F.Cu at (82.1, 246.5)
- added REF**: washer, kbd:washer, F.Cu at (82.1, 255.5)
- added REF**: L_case_parts, kbd:L_case_parts, F.Cu at (286.0, 52.0)
- added REF**: washer, kbd:washer, F.Cu at (90.1, 246.4)
- added REF**: washer, kbd:washer, F.Cu at (41.0, 273.2)
- added REF**: washer, kbd:washer, F.Cu at (33.0, 282.3)
- added REF**: washer, kbd:washer, F.Cu at (41.0, 282.2)
- added REF**: washer, kbd:washer, F.Cu at (33.0, 273.3)
- added REF**: washer, kbd:washer, F.Cu at (74.0, 264.2)
- added REF**: washer, kbd:washer, F.Cu at (74.0, 282.2)
- added REF**: washer, kbd:washer, F.Cu at (66.0, 282.3)
- added REF**: washer, kbd:washer, F.Cu at (66.0, 273.3)
- added REF**: washer, kbd:washer, F.Cu at (74.0, 273.2)
- added REF**: L_case_parts, kbd:L_case_parts, B.Cu at (299.0, 20.0)
- added REF**: washer, kbd:washer, F.Cu at (66.0, 264.3)
- added REF**: washer, kbd:washer, F.Cu at (74.0, 255.2)
- added REF**: washer, kbd:washer, F.Cu at (66.0, 246.3)
- added REF**: washer, kbd:washer, F.Cu at (66.0, 255.3)
- added REF**: washer, kbd:washer, F.Cu at (74.0, 219.2)
- added REF**: washer, kbd:washer, F.Cu at (74.0, 237.2)
- added REF**: washer, kbd:washer, F.Cu at (66.0, 237.3)
- added REF**: washer, kbd:washer, F.Cu at (66.0, 228.3)
- added REF**: washer, kbd:washer, F.Cu at (74.0, 228.2)
- added REF**: washer, kbd:washer, F.Cu at (74.0, 246.2)
- added REF**: L_case_parts, kbd:L_case_parts, B.Cu at (305.0, 14.0)
- added REF**: washer, kbd:washer, F.Cu at (66.0, 219.3)
- added REF**: washer, kbd:washer, F.Cu at (58.0, 282.2)
- added REF**: washer, kbd:washer, F.Cu at (50.0, 273.3)
- added REF**: washer, kbd:washer, F.Cu at (50.0, 282.3)
- added REF**: washer, kbd:washer, F.Cu at (58.0, 246.2)
- added REF**: washer, kbd:washer, F.Cu at (58.0, 264.2)
- added REF**: washer, kbd:washer, F.Cu at (50.0, 264.3)
- added REF**: washer, kbd:washer, F.Cu at (50.0, 255.3)
- added REF**: washer, kbd:washer, F.Cu at (58.0, 255.2)
- added REF**: washer, kbd:washer, F.Cu at (58.0, 273.2)
- added REF**: L_case_parts, kbd:L_case_parts, B.Cu at (302.0, 17.0)
- added REF**: washer, kbd:washer, F.Cu at (50.0, 246.3)
- added REF**: washer, kbd:washer, F.Cu at (58.0, 237.2)
- added REF**: washer, kbd:washer, F.Cu at (50.0, 228.3)
- added REF**: washer, kbd:washer, F.Cu at (50.0, 237.3)
- added REF**: washer, kbd:washer, F.Cu at (58.0, 201.2)
- added REF**: washer, kbd:washer, F.Cu at (58.0, 219.2)
- added REF**: washer, kbd:washer, F.Cu at (50.0, 219.3)
- added REF**: washer, kbd:washer, F.Cu at (50.0, 210.3)
- added REF**: washer, kbd:washer, F.Cu at (58.0, 210.2)
- added REF**: washer, kbd:washer, F.Cu at (58.0, 228.2)
- added REF**: L_case_parts, kbd:L_case_parts, F.Cu at (26.0, 216.0)
- added REF**: washer, kbd:washer, F.Cu at (50.0, 201.3)
- added REF**: washer, kbd:washer, F.Cu at (41.0, 264.2)
- added REF**: washer, kbd:washer, F.Cu at (33.0, 255.3)
- added REF**: washer, kbd:washer, F.Cu at (33.0, 264.3)
- added REF**: washer, kbd:washer, F.Cu at (41.0, 228.2)
- added REF**: washer, kbd:washer, F.Cu at (41.0, 246.2)
- added REF**: washer, kbd:washer, F.Cu at (33.0, 246.3)
- added REF**: washer, kbd:washer, F.Cu at (33.0, 237.3)
- added REF**: washer, kbd:washer, F.Cu at (41.0, 237.2)
- added REF**: washer, kbd:washer, F.Cu at (41.0, 255.2)
- added REF**: L_case_parts, kbd:L_case_parts, F.Cu at (131.0, 218.0)
- added REF**: washer, kbd:washer, F.Cu at (33.0, 228.3)
- added REF**: washer, kbd:washer, F.Cu at (41.0, 219.2)
- added REF**: washer, kbd:washer, F.Cu at (33.0, 219.3)
- added REF**: washer, kbd:washer, F.Cu at (41.0, 210.2)
- added REF**: washer, kbd:washer, F.Cu at (33.0, 210.3)
- added REF**: washer, kbd:washer, F.Cu at (41.0, 201.2)
- added REF**: washer, kbd:washer, F.Cu at (33.0, 201.3)
- added REF**: washer, kbd:washer, F.Cu at (41.0, 192.2)
- added REF**: washer, kbd:washer, F.Cu at (33.0, 192.3)
- added REF**: washer, kbd:washer, F.Cu at (41.0, 183.2)
- added REF**: L_case_parts, kbd:L_case_parts, F.Cu at (143.0, 255.0)
- added REF**: washer, kbd:washer, F.Cu at (33.0, 183.3)
- added REF**: L_case_parts, kbd:L_case_parts, F.Cu at (33.0, 253.0)
