File: pcb/gbr/fan.kicad_pcb (KiCad board)
At the start: 2 copper layers, 706.1 x 736.6 mm, 86 parts, among them J1 MJ-4PP-9, SW1 SW_PUSH-kbd, SW10 SW_PUSH-kbd, SW11 SW_PUSH-kbd, SW12 SW_PUSH-kbd, SW13 SW_PUSH-kbd, SW14 SW_PUSH-kbd, SW15 SW_PUSH-kbd, SW16 SW_PUSH-kbd, SW17 SW_PUSH-kbd, SW18 SW_PUSH-kbd, SW19 SW_PUSH-kbd, SW2 SW_PUSH-kbd, SW20 SW_PUSH-kbd, SW21 SW_PUSH-kbd, SW22 SW_PUSH-kbd, SW23 SW_PUSH-kbd, SW24 SW_PUSH-kbd, SW25 SW_PUSH-kbd, SW26 SW_PUSH-kbd, SW27 SW_PUSH-kbd, SW28 SW_PUSH-kbd, SW29 SW_PUSH-kbd, SW3 SW_PUSH-kbd, SW30 SW_PUSH-kbd, SW31 SW_PUSH-kbd, SW32 SW_PUSH-kbd, SW33 SW_PUSH-kbd, SW34 SW_PUSH-kbd, SW35 SW_PUSH-kbd, SW36 SW_PUSH-kbd, SW37 SW_PUSH-kbd, SW38 SW_PUSH-kbd, SW39 SW_PUSH-kbd, SW4 SW_PUSH-kbd, SW40 SW_PUSH-kbd, SW41 SW_PUSH, SW5 SW_PUSH-kbd, SW6 SW_PUSH-kbd, SW7 SW_PUSH-kbd, SW8 SW_PUSH-kbd, SW9 SW_PUSH-kbd, U1 BluePill_STM32F103C, U2 BluePill_STM32F103C

Commit message: fan74のPCBが一応完成した
Parts:
- moved Ref** 372.0 mm to (226.4, 448.5)
- moved Ref** 372.0 mm to (96.2, 504.0)
- moved Ref** 372.0 mm to (150.8, 401.4)
- moved Ref** 372.0 mm to (230.9, 487.7)
- moved Ref** 372.0 mm to (39.5, 523.7)
- moved Ref** 372.0 mm to (226.4, 535.7)
- moved Ref** 372.0 mm to (194.6, 408.0)
- moved Ref** 372.0 mm to (89.4, 408.4)
- moved Ref** 372.0 mm to (165.7, 504.6)
- moved Ref** 372.0 mm to (152.3, 441.7)
- moved Ref** 372.0 mm to (89.6, 450.0)
- moved Ref** 372.0 mm to (32.6, 443.4)
- moved Ref** 372.0 mm to (28.5, 481.1)
Other:
- board size 706.1 x 736.6 mm -> 347.6 x 529.6 mm
