File: pcb/fan.kicad_pcb (KiCad board)
At the start: 2 copper layers, 706.1 x 736.6 mm, 86 parts, among them J1 MJ-4PP-9, SW1 SW_PUSH-kbd, SW10 SW_PUSH-kbd, SW11 SW_PUSH-kbd, SW12 SW_PUSH-kbd, SW13 SW_PUSH-kbd, SW14 SW_PUSH-kbd, SW15 SW_PUSH-kbd, SW16 SW_PUSH-kbd, SW17 SW_PUSH-kbd, SW18 SW_PUSH-kbd, SW19 SW_PUSH-kbd, SW2 SW_PUSH-kbd, SW20 SW_PUSH-kbd, SW21 SW_PUSH-kbd, SW22 SW_PUSH-kbd, SW23 SW_PUSH-kbd, SW24 SW_PUSH-kbd, SW25 SW_PUSH-kbd, SW26 SW_PUSH-kbd, SW27 SW_PUSH-kbd, SW28 SW_PUSH-kbd, SW29 SW_PUSH-kbd, SW3 SW_PUSH-kbd, SW30 SW_PUSH-kbd, SW31 SW_PUSH-kbd, SW32 SW_PUSH-kbd, SW33 SW_PUSH-kbd, SW34 SW_PUSH-kbd, SW35 SW_PUSH-kbd, SW36 SW_PUSH-kbd, SW37 SW_PUSH-kbd, SW38 SW_PUSH-kbd, SW39 SW_PUSH-kbd, SW4 SW_PUSH-kbd, SW40 SW_PUSH-kbd, SW41 SW_PUSH, SW5 SW_PUSH-kbd, SW6 SW_PUSH-kbd, SW7 SW_PUSH-kbd, SW8 SW_PUSH-kbd, SW9 SW_PUSH-kbd, U1 BluePill_STM32F103C, U2 BluePill_STM32F103C

Commit message: fan74のケースを作成
Parts:
- removed R10, R11, R9: 10K, keyboard_parts:R_1608_rev2
- removed the Ref** at (944.5, 30.3)
- removed the Ref** at (994.4, 145.6)
- removed the Ref** at (1099.6, 146.0)
- removed the Ref** at (933.5, 72.9)
- removed the Ref** at (937.6, 110.6)
- removed the Ref** at (-143.6, 409.5)
- removed the Ref** at (-273.8, 465.0)
- removed the Ref** at (-219.2, 362.4)
- removed the Ref** at (-139.1, 448.7)
- removed the Ref** at (-330.5, 484.7)
- removed the Ref** at (-143.6, 496.7)
- removed the Ref** at (1131.4, 105.5)
- removed the Ref** at (-175.4, 369.0)
- removed the Ref** at (-280.6, 369.4)
- removed the Ref** at (-204.3, 465.6)
- removed the Ref** at (-217.7, 402.7)
- removed the Ref** at (-280.4, 411.0)
- removed the Ref** at (-337.4, 404.4)
- removed the Ref** at (-341.5, 442.1)
- removed the Ref** at (76.6, 64.0)
- removed the Ref** at (1001.2, 50.0)
- removed the Ref** at (139.3, 55.7)
- removed the Ref** at (152.7, 118.6)
- removed the Ref** at (76.4, 22.4)
- removed the Ref** at (181.6, 22.0)
- removed the Ref** at (213.4, 149.7)
- removed the Ref** at (26.5, 137.7)
- removed the Ref** at (217.9, 101.7)
- removed the Ref** at (137.8, 15.4)
- removed the Ref** at (83.2, 118.0)
- removed the Ref** at (213.4, 62.5)
- removed the Ref** at (1055.8, 152.6)
- removed the Ref** at (1070.7, 49.4)
- removed the Ref** at (1057.3, 112.3)
- removed the Ref** at (1135.9, 66.3)
- removed the Ref** at (1131.4, 18.3)
- removed the Ref** at (994.6, 104.0)
- removed U2: BluePill_STM32F103C, BluePill_breakouts:BluePill_STM32F103C
- added R1: 10K, keyboard_parts:R_1608_rev2, F.Cu at (204.5, 41.0)
- added R2: 10K, keyboard_parts:R_1608_rev2, F.Cu at (205.5, 62.1)
- added Ref**: Val**, kbd:HOLE, F.Cu at (25.7, 138.3)
- added Ref**: Val**, kbd:HOLE, F.Cu at (212.0, 73.5)
- added Ref**: Val**, kbd:HOLE, F.Cu at (137.8, 15.4)
- added Ref**: Val**, kbd:HOLE, F.Cu at (83.2, 120.9)
- added Ref**: Val**, kbd:HOLE, F.Cu at (76.6, 64.0)
- added Ref**: Val**, kbd:HOLE, F.Cu at (139.3, 55.7)
- added Ref**: Val**, kbd:HOLE, F.Cu at (152.6, 118.6)
- added Ref**: Val**, kbd:HOLE, F.Cu at (76.3, 22.3)
- added Ref**: Val**, kbd:HOLE, F.Cu at (181.2, 22.3)
- added Ref**: Val**, kbd:HOLE, F.Cu at (213.8, 149.7)
- U1: footprint BluePill_breakouts:BluePill_STM32F103C -> BluePill_breakouts:BluePill_STM32F103C_0.9_Double
- moved J1 49.0 mm to (209.0, 49.0), turned to 0 degrees
- moved SW41 42.1 mm to (209.2, 62.5), turned to 90 degrees
- moved Ref** 3.67 mm to (14.6, 98.7)
- moved Ref** 2.87 mm to (20.4, 60.1)
- moved U1 0.47 mm to (191.4, 59.1), turned to 0 degrees
- moved SW2 0.07 mm to (31.1, 77.2)
- moved SW29 0.07 mm to (123.6, 83.6)
- moved SW38 0.07 mm to (168.3, 67.1)
- moved SW10 0.07 mm to (25.4, 91.6)
- moved SW14 0.07 mm to (64.1, 101.3)
- moved SW16 0.07 mm to (88.0, 29.0)
- moved SW9 0.07 mm to (48.2, 114.1)
- moved SW36 0.07 mm to (167.2, 27.8)
- moved SW40 0.07 mm to (209.9, 139.5)
- moved SW28 0.07 mm to (128.9, 63.9)
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Connections:
- J1 pad B: Tx -> Rx
- U1 pad 1: (no net) -> Net-(U1-Pad1)
- U1 pad 15: (no net) -> Net-(U1-Pad15)
- U1 pad 16: (no net) -> Net-(U1-Pad16)
- U1 pad 2: (no net) -> Net-(U1-Pad2)
- U1 pad 21: (no net) -> Net-(U1-Pad21)
- U1 pad 22: (no net) -> Net-(U1-Pad22)
- U1 pad 23: (no net) -> Net-(U1-Pad23)
- U1 pad 24: (no net) -> Net-(U1-Pad24)
- U1 pad 25: (no net) -> Net-(U1-Pad25)
- U1 pad 26: Tx -> Rx
- U1 pad 28: (no net) -> Net-(U1-Pad28)
- U1 pad 29: (no net) -> Net-(U1-Pad29)
- U1 pad 3: (no net) -> Net-(U1-Pad3)
- U1 pad 30: (no net) -> Net-(U1-Pad30)
- U1 pad 31: (no net) -> Net-(U1-Pad31)
- U1 pad 32: (no net) -> Net-(U1-Pad32)
- U1 pad 38: (no net) -> Net-(U1-Pad38)
- U1 pad 4: (no net) -> Net-(U1-Pad4)
- U1 pad 7: (no net) -> Net-(U1-Pad7)
- U1 pad 8: (no net) -> Net-(U1-Pad8)
Routing:
- net Tx: track 64.0 -> 0.00 mm
- net Rx: track 23.1 -> 76.5 mm
- net VCC: track 138.7 -> 101.3 mm, vias 1 -> 3
- net GND: track 46.1 -> 69.2 mm, vias 205 -> 104
- net Net-(U1-Pad1): track 0.00 -> 17.5 mm
- net Net-(U1-Pad8): track 0.00 -> 17.5 mm
- net Net-(U1-Pad7): track 0.00 -> 17.5 mm
- net Net-(U1-Pad4): track 0.00 -> 17.5 mm
- net Net-(U1-Pad3): track 0.00 -> 17.5 mm
- net Net-(U1-Pad2): track 0.00 -> 17.5 mm
- net Net-(U1-Pad16): track 0.00 -> 17.5 mm
- net Net-(U1-Pad15): track 0.00 -> 17.5 mm
- net Net-(U1-Pad28): track 0.00 -> 14.1 mm
- net Net-(U1-Pad21): track 0.00 -> 14.1 mm
- net Net-(U1-Pad32): track 0.00 -> 14.1 mm
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Other:
- board size 706.1 x 736.6 mm -> 212.8 x 143.6 mm
