File: pcb/fan.kicad_pcb (KiCad board)
At the start: 2 copper layers, 212.8 x 143.6 mm, 57 parts, among them J1 MJ-4PP-9, SW1 SW_PUSH-kbd, SW10 SW_PUSH-kbd, SW11 SW_PUSH-kbd, SW12 SW_PUSH-kbd, SW13 SW_PUSH-kbd, SW14 SW_PUSH-kbd, SW15 SW_PUSH-kbd, SW16 SW_PUSH-kbd, SW17 SW_PUSH-kbd, SW18 SW_PUSH-kbd, SW19 SW_PUSH-kbd, SW2 SW_PUSH-kbd, SW20 SW_PUSH-kbd, SW21 SW_PUSH-kbd, SW22 SW_PUSH-kbd, SW23 SW_PUSH-kbd, SW24 SW_PUSH-kbd, SW25 SW_PUSH-kbd, SW26 SW_PUSH-kbd, SW27 SW_PUSH-kbd, SW28 SW_PUSH-kbd, SW29 SW_PUSH-kbd, SW3 SW_PUSH-kbd, SW30 SW_PUSH-kbd, SW31 SW_PUSH-kbd, SW32 SW_PUSH-kbd, SW33 SW_PUSH-kbd, SW34 SW_PUSH-kbd, SW35 SW_PUSH-kbd, SW36 SW_PUSH-kbd, SW37 SW_PUSH-kbd, SW38 SW_PUSH-kbd, SW39 SW_PUSH-kbd, SW4 SW_PUSH-kbd, SW40 SW_PUSH-kbd, SW41 SW_PUSH, SW5 SW_PUSH-kbd, SW6 SW_PUSH-kbd, SW7 SW_PUSH-kbd, SW8 SW_PUSH-kbd, SW9 SW_PUSH-kbd, U1 BluePill_STM32F103C

Commit message: 異種面付けしてみた がしないで3枚注文してもトントンだったので 普通に発注する予定
Parts:
- removed the Ref** at (25.7, 138.3)
- removed the Ref** at (212.0, 73.5)
- removed the Ref** at (137.8, 15.4)
- removed the Ref** at (76.6, 64.0)
- removed the Ref** at (139.3, 55.7)
- removed the Ref** at (152.6, 118.6)
- removed the Ref** at (76.3, 22.3)
- removed the Ref** at (181.2, 22.3)
- removed the Ref** at (213.8, 149.7)
- added J2: Conn_01x01_Female, Connector_Pin:Pin_D1.0mm_L10.0mm, F.Cu at (61.9, 76.0)
- added J3: Conn_01x01_Female, Connector_Pin:Pin_D1.0mm_L10.0mm, F.Cu at (65.1, 76.5)
- added Ref**: Val**, kbd:HOLE, F.Cu at (50.5, 77.1)
- added Ref**: Val**, kbd:HOLE, F.Cu at (86.5, 40.6)
- added Ref**: Val**, kbd:HOLE, F.Cu at (28.4, 114.8)
- added Ref**: Val**, kbd:HOLE, F.Cu at (151.3, 226.9)
- added Ref**: Val**, kbd:HOLE, F.Cu at (77.0, 176.0)
- added Ref**: Val**, kbd:HOLE, F.Cu at (68.7, 113.3)
- added Ref**: Val**, kbd:HOLE, F.Cu at (131.6, 100.0)
- added Ref**: Val**, kbd:HOLE, F.Cu at (35.3, 176.3)
- added Ref**: Val**, kbd:HOLE, F.Cu at (162.7, 38.8)
- moved Ref** 180.0 mm to (73.1, 232.2), turned to 90 degrees
- moved SW1 172.2 mm to (65.7, 221.4), turned to 125 degrees
- moved SW5 171.6 mm to (79.2, 228.6), turned to 306 degrees
- moved Ref** 169.0 mm to (111.7, 237.0), turned to 90 degrees
- moved SW6 162.3 mm to (54.8, 203.9), turned to 117 degrees
- moved SW10 157.1 mm to (104.6, 227.2), turned to 312 degrees
- moved SW2 155.9 mm to (90.2, 221.5), turned to 127 degrees
- moved SW11 152.5 mm to (46.7, 184.7), turned to 108 degrees
- moved R1 150.7 mm to (54.0, 48.1), turned to 90 degrees
- moved J1 147.1 mm to (62.0, 43.6), turned to 90 degrees
- moved SW15 146.2 mm to (127.8, 223.0), turned to 318 degrees
- moved SW16 143.2 mm to (42.0, 164.6), turned to 100 degrees
- moved SW7 143.2 mm to (78.6, 205.3), turned to 123 degrees
- moved SW3 140.2 mm to (112.1, 216.7), turned to 132 degrees
- moved SW4 139.9 mm to (141.3, 218.4), turned to 138 degrees
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Routing:
- net Net-(J3-Pad1): track 17.5 -> 25.4 mm
- net Net-(J2-Pad1): track 17.5 -> 25.2 mm
- net col07: track 314.5 -> 312.8 mm
- net GND: vias 104 -> 316
- net (no net): vias 0 -> 2
Other:
- board size 212.8 x 143.6 mm -> 420 x 250 mm

Commit message: 天板 底板を作成 したものの、あと数ミリ小さくする予定
Parts:
- removed the Ref** at (86.5, 40.6)
- removed the Ref** at (28.4, 114.8)
- removed the Ref** at (151.3, 226.9)
- removed the Ref** at (77.0, 176.0)
- removed the Ref** at (68.7, 113.3)
- removed the Ref** at (131.6, 100.0)
- removed the Ref** at (35.3, 176.3)
- removed the Ref** at (162.7, 38.8)
- added Ref**: Val**, kbd:HOLE, F.Cu at (66.0, 54.0)
- added Ref**: Val**, kbd:HOLE, F.Cu at (203.2, 139.7)
- added Ref**: Val**, kbd:HOLE, F.Cu at (201.4, 63.5)
- added Ref**: Val**, kbd:HOLE, F.Cu at (142.0, 108.6)
- added Ref**: Val**, kbd:HOLE, F.Cu at (65.7, 12.3)
- added Ref**: Val**, kbd:HOLE, F.Cu at (127.1, 5.65)
- added Ref**: Val**, kbd:HOLE, F.Cu at (15.1, 128.3)
- added Ref**: Val**, kbd:HOLE, F.Cu at (128.7, 45.7)
- moved Ref** 192.8 mm to (9.80, 50.1), turned to 0 degrees
- moved SW5 184.6 mm to (13.4, 56.2), turned to 216 degrees
- moved SW1 184.4 mm to (20.6, 42.7), turned to 35 degrees
- moved Ref** 182.7 mm to (5.00, 88.7), turned to 0 degrees
- moved SW6 173.0 mm to (38.1, 31.8), turned to 27 degrees
- moved SW10 171.1 mm to (14.8, 81.6), turned to 222 degrees
- moved SW2 169.3 mm to (20.5, 67.2), turned to 37 degrees
- moved SW11 161.4 mm to (57.3, 23.7), turned to 18 degrees
- moved SW15 160.7 mm to (19.0, 104.8), turned to 228 degrees
- moved SW7 155.5 mm to (36.7, 55.6), turned to 33 degrees
- moved SW4 154.5 mm to (23.6, 118.3), turned to 48 degrees
- moved SW3 154.4 mm to (25.3, 89.1), turned to 42 degrees
- moved SW16 149.9 mm to (77.4, 19.0), turned to 10 degrees
- moved SW12 141.5 mm to (55.3, 45.9), turned to 22 degrees
- moved SW21 141.3 mm to (96.8, 16.2), turned to 6 degrees
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Routing:
- net GND: vias 316 -> 338
Other:
- board size 420 x 250 mm -> 212.8 x 143.6 mm
- board text added: "Fan74 v1.0 Designed by H&C 20200314"
- board text removed: "Fan74 v1.0 Designed by @xcd0 20200314"
